File: MVSC2.kicad_pcb (KiCad board)
At the start: 4 copper layers, 88.1 x 95.6 mm, 340 parts, among them J1 USB_C-SIGNAL, J10 PWM3_OUT, J11 PWM_IN, J12 EXP-1, J13 Exp2-smd, J14 EXP-3, J15 EXP-2, J16 ADC0, J17 ESTP0, J18 ESTP1, J19 ESTP2, J2 SERV2, J20 ESTP3, J21 ESTP4, J22 ESTP5, J23 POWER, J24 CaEx2, J25 SERV0, J26 SERV1, J27 CaEx2, J28 CaEx3, J29 ADC1, J3 EXP0, J30 HSES, J31 HSES, J32 HSES, J33 CaEx3, J34 SERV3, J35 SERV4, J36 SERV5, J37 EXP-SERVO, J38 I2C, J39 UART_pin, J4 EXP1, J40 UART, J41 I2C_pin, J42 I2C, J5 UART, J6 PWM0_OUT, J7 PWM1_OUT, J8 Exp1-pin, J9 PWM2_OUT, P1 STP0, P2 STP2, P3 STP4, P4 STP1, P5 STP3, P6 STP5, P7 CaEx4, P8 CaEx4, Q1 AO3400A, Q10 AO3400A, Q2 AO3400A, Q3 AO3400A, Q4 AO3400A, Q5 AO3400A, Q6 AO3400A, SW1 SKRKAEE020, SW2 SKRKAEE020, U1 XC6206P332MR, U10 TMC2208-LA-T, U11 TMC2208-LA-T, U12 TMC2208-LA-T, U3 STM32F411RCT6, U4 CH912LSR, U5 TMC2208-LA-T, U6 TMC2208-LA-T, U7 TMC2208-LA-T, U8 CH912LSR, U9 CH912LSR, Y1 25MHZ 12pF, Y2 32.768KHz 12.5pF

Commit message: working
Parts:
- removed C120, C121, C2, C4: 4.7uF 10V, Capacitor_SMD:C_0402_1005Metric
- removed J12: EXP-1, Connector_FFC-FPC:Hirose_FH12-20S-0.5SH_1x20-1MP_P0.50mm_Horizontal
- removed J13: Exp2-smd, Connector_PinHeader_2.00mm:PinHeader_1x11_P2.00mm_Horizontal
- removed J14: EXP-3, Connector_FFC-FPC:Hirose_FH12-20S-0.5SH_1x20-1MP_P0.50mm_Horizontal
- removed J15: EXP-2, Connector_FFC-FPC:Hirose_FH12-20S-0.5SH_1x20-1MP_P0.50mm_Horizontal
- removed J24, J27: CaEx2, Connector_JST:JST_PH_B2B-PH-K_1x02_P2.00mm_Vertical
- removed J28, J33: CaEx3, Connector_JST:JST_PH_B3B-PH-K_1x03_P2.00mm_Vertical
- removed J34: SERV3, Connector_JST:JST_PH_B3B-PH-K_1x03_P2.00mm_Vertical
- removed J35: SERV4, Connector_JST:JST_PH_B3B-PH-K_1x03_P2.00mm_Vertical
- removed J36: SERV5, Connector_JST:JST_PH_B3B-PH-K_1x03_P2.00mm_Vertical
- removed J37: EXP-SERVO, Connector_FFC-FPC:Hirose_FH12-20S-0.5SH_1x20-1MP_P0.50mm_Horizontal
- removed J38, J42: I2C, Connector_FFC-FPC:Hirose_FH12-6S-0.5SH_1x06-1MP_P0.50mm_Horizontal
- removed J39: UART_pin, Connector_PinHeader_2.54mm:PinHeader_1x04_P2.54mm_Vertical
- removed J40, J5: UART, Connector_FFC-FPC:Hirose_FH12-6S-0.5SH_1x06-1MP_P0.50mm_Horizontal
- removed J41: I2C_pin, Connector_PinHeader_2.54mm:PinHeader_1x04_P2.54mm_Vertical
- removed J8: Exp1-pin, Connector_PinHeader_2.54mm:PinHeader_1x11_P2.54mm_Vertical
- removed JP1, JP2, JP3, JP4, JP5, JP6, JP7, JP8: SJ_O, Jumper:SolderJumper-2_P1.3mm_Open_RoundedPad1.0x1.5mm
- removed P7, P8: CaEx4, Connector_JST:JST_PH_B4B-PH-K_1x04_P2.00mm_Vertical
- removed R13, R14, R15, R16: 4.7k, Resistor_SMD:R_0402_1005Metric
- removed mouse-bite-2mm-slot (x32): VAL**, Panelization:mouse-bite-2mm-slot
- added P9: UART, Connector_JST:JST_PH_B4B-PH-K_1x04_P2.00mm_Vertical, F.Cu at (182.8, 155.0)
- added REF**: ToolingHole, MountingHole:MountingHole_3.2mm_M3, F.Cu at (178.0, 78.0)
- added REF**: MountingHole_3.2mm_M3, MountingHole:MountingHole_3.2mm_M3, F.Cu at (165.0, 130.0)
- added REF**: MountingHole_3.2mm_M3, MountingHole:MountingHole_3.2mm_M3, F.Cu at (137.4, 130.0)
- added REF**: MountingHole_3.2mm_M3, MountingHole:MountingHole_3.2mm_M3, F.Cu at (165.0, 150.0)
- added REF**: MountingHole_3.2mm_M3, MountingHole:MountingHole_3.2mm_M3, F.Cu at (137.4, 150.0)
- added REF**: MountingHole_3.2mm_M3, MountingHole:MountingHole_3.2mm_M3, F.Cu at (155.4, 115.2)
- added REF**: MountingHole_3.2mm_M3, MountingHole:MountingHole_3.2mm_M3, F.Cu at (175.4, 78.8)
- added REF**: MountingHole_3.2mm_M3, MountingHole:MountingHole_3.2mm_M3, F.Cu at (155.4, 78.8)
- added REF**: ToolingHole, MountingHole:MountingHole_3.2mm_M3, F.Cu at (180.0, 78.0)
- added REF**: ToolingHole, MountingHole:MountingHole_3.2mm_M3, F.Cu at (176.6, 166.0)
- added REF**: MountingHole_3.2mm_M3, MountingHole:MountingHole_3.2mm_M3, F.Cu at (144.7, 119.3)
- added REF**: MountingHole_3.2mm_M3, MountingHole:MountingHole_3.2mm_M3, F.Cu at (144.7, 109.6)
- added REF**: MountingHole_3.2mm_M3, MountingHole:MountingHole_3.2mm_M3, F.Cu at (144.7, 99.8)
- added REF**: MountingHole_3.2mm_M3, MountingHole:MountingHole_3.2mm_M3, F.Cu at (144.7, 90.0)
- J2: value SERV2 -> EXP0; footprint Connector_JST:JST_PH_B3B-PH-K_1x03_P2.00mm_Vertical -> Connector_PinHeader_2.00mm:PinHeader_1x08_P2.00mm_Vertical; moved to F.Cu
- J3: value EXP0 -> EXP1; footprint Connector_FFC-FPC:Hirose_FH12-20S-0.5SH_1x20-1MP_P0.50mm_Horizontal -> Connector_PinHeader_2.00mm:PinHeader_1x08_P2.00mm_Vertical
- J4: value EXP1 -> EXPB; footprint Connector_FFC-FPC:Hirose_FH12-20S-0.5SH_1x20-1MP_P0.50mm_Horizontal -> Connector_PinHeader_2.00mm:PinHeader_1x08_P2.00mm_Vertical
- moved R2 70.3 mm to (184.4, 85.3), turned to 90 degrees
- moved R26 69.1 mm to (184.5, 105.9), turned to 90 degrees
- moved R11 65.9 mm to (183.1, 88.5), turned to 180 degrees
- moved D6 65.7 mm to (181.4, 109.7), turned to 180 degrees
- moved Q3 63.8 mm to (181.0, 85.3), turned to 180 degrees
- moved Q10 61.9 mm to (181.0, 105.4), turned to 180 degrees
- moved D5 60.8 mm to (180.9, 90.3), turned to 0 degrees
- moved D9 60.6 mm to (181.3, 100.3), turned to 270 degrees
- moved R39 56.5 mm to (179.4, 95.3), turned to 90 degrees
- moved C26 56.5 mm to (179.4, 97.5), turned to 90 degrees
- moved J10 55.8 mm to (176.4, 108.7), turned to 180 degrees
- moved J7 53.6 mm to (175.4, 85.3), turned to 270 degrees
- moved J9 52.0 mm to (176.4, 103.2), turned to 180 degrees
- moved J29 50.4 mm to (176.4, 96.7), turned to 180 degrees
- moved J4 50.3 mm to (170.2, 115.2), turned to 90 degrees
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Connections:
- net GND_E3 renamed GND_EB
- net V_PWM_E3 renamed V_PWM_EB
- C25 pad 1: ADCGND_E3 -> GND_EB_ADC
- C26 pad 1: ADCGND_E3 -> GND_EB_ADC
- J16 pad 1: ADCGND_E3 -> GND_EB_ADC
- J2 pad 1: PWM0_E0 -> GND
- J2 pad 2: GND_E0 -> Net-(J2-Pad2)
- J2 pad 3: V_SERVO_E0 -> Net-(J2-Pad3)
- J29 pad 1: ADCGND_E3 -> GND_EB_ADC
- J3 pad 2: GND -> Net-(J3-Pad2)
- J3 pad 3: GND -> Net-(J3-Pad3)
- J3 pad 4: V_SERVO -> Net-(J3-Pad4)
- J3 pad 5: V_SERVO -> Net-(J3-Pad5)
- J3 pad 6: V_SERVO -> Net-(J3-Pad6)
- J3 pad 7: +3V3 -> Net-(J3-Pad7)
- J3 pad 8: Net-(J3-Pad8) -> V_SERVO
- J4 pad 1: GND -> GND_EB_ADC
- J4 pad 2: GND -> PWM3_E3
- J4 pad 3: GND -> PWM2_E3
- J4 pad 4: V_SERVO -> ADC1
- J4 pad 5: V_SERVO -> ADC0
- J4 pad 6: V_SERVO -> PWM1_E3
- J4 pad 7: +3V3 -> PWM0_E3
- J4 pad 8: Net-(J4-Pad8) -> 3V3_EB
- R31 pad 2: 3v3_E3 -> 3V3_EB
- R32 pad 2: Net-(J3-Pad8) -> Net-(J3-Pad7)
- R33 pad 2: Net-(J3-Pad9) -> Net-(J3-Pad6)
- R34 pad 2: Net-(J3-Pad10) -> Net-(J3-Pad5)
- R35 pad 2: Net-(J3-Pad11) -> Net-(J3-Pad4)
- R36 pad 2: Net-(J3-Pad12) -> Net-(J3-Pad3)
- R37 pad 2: Net-(J3-Pad13) -> Net-(J3-Pad2)
- R38 pad 2: Net-(J4-Pad9) -> Net-(J2-Pad7)
- R39 pad 2: 3v3_E3 -> 3V3_EB
- R40 pad 2: Net-(J4-Pad10) -> Net-(J2-Pad5)
- R41 pad 2: Net-(J4-Pad11) -> Net-(J2-Pad4)
- R42 pad 2: Net-(J4-Pad8) -> Net-(J2-Pad6)
- R43 pad 2: Net-(J4-Pad12) -> Net-(J2-Pad3)
- R44 pad 2: Net-(J4-Pad13) -> Net-(J2-Pad2)
Routing:
- net 3v3_E3: track 87.2 -> 0.00 mm, vias 3 -> 0
- net 3V3_EB: track 0.00 -> 75.7 mm, vias 0 -> 3
- net Net-(J2-Pad2): track 0.00 -> 53.1 mm, vias 0 -> 2
- net GND_EB_ADC: track 0.00 -> 51.1 mm, vias 0 -> 1
- net ADCGND_E3: track 51.6 -> 0.88 mm, vias 1 -> 0
- net Net-(J2-Pad3): track 0.00 -> 49.2 mm, vias 0 -> 2
- net Net-(J4-Pad13): track 46.9 -> 0.00 mm, vias 2 -> 0
- net Net-(J4-Pad12): track 45.8 -> 0.00 mm, vias 2 -> 0
- net 3v3_E0: track 40.1 -> 0.00 mm
- net Net-(J2-Pad4): track 0.00 -> 37.8 mm, vias 0 -> 2
- net Net-(J4-Pad11): track 37.7 -> 0.00 mm, vias 2 -> 0
- net Net-(J13-Pad6): track 36.7 -> 0.00 mm, vias 2 -> 0
- net Net-(J13-Pad7): track 35.8 -> 0.00 mm
- net Net-(J13-Pad5): track 35.8 -> 0.00 mm
- net Net-(J2-Pad5): track 0.00 -> 33.6 mm, vias 0 -> 2
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- added copper zone on F.Cu, net GND_EB_ADC
- removed copper zone on F.Cu, net (none)
- removed copper zone on B.Cu, net GND_E0
- removed copper zone on F.Cu, net GND_E0
- removed copper zone on In1.Cu, net GND_E0
- removed copper zone on In2.Cu, net GND_E0
- removed copper zone on F.Cu, net Net-(C120-Pad1)
- removed copper zone on F.Cu, net Net-(C121-Pad1)
- removed copper zone on F.Cu, net Net-(C27-Pad2)
- removed copper zone on F.Cu, net Net-(C52-Pad2)
- removed copper zone on F.Cu, net Net-(C68-Pad2)
- removed copper zone on F.Cu, net Net-(D3-Pad2)
- removed copper zone on F.Cu, net Net-(J24-Pad1)
- removed copper zone on B.Cu, net Net-(J24-Pad2)
- removed copper zone on In1.Cu, net Net-(J24-Pad2)
- removed copper zone on In2.Cu, net Net-(J24-Pad2)
- removed copper zone on In2.Cu, net Net-(J28-Pad1)
- removed copper zone on B.Cu, net Net-(J28-Pad3)
- removed copper zone on In1.Cu, net Net-(J28-Pad3)
- removed copper zone on B.Cu, net Net-(J39-Pad2)
- removed copper zone on F.Cu, net Net-(J39-Pad2)
- removed copper zone on In1.Cu, net Net-(J39-Pad2)
- removed copper zone on In2.Cu, net Net-(J39-Pad2)
- removed copper zone on B.Cu, net Net-(J41-Pad1)
- removed copper zone on F.Cu, net Net-(J41-Pad1)
- removed copper zone on In1.Cu, net Net-(J41-Pad1)
- removed copper zone on In2.Cu, net Net-(J41-Pad1)
- removed copper zone on In1.Cu, net Net-(P7-Pad1)
- removed copper zone on B.Cu, net Net-(P7-Pad2)
- removed copper zone on In2.Cu, net Net-(P7-Pad4)
- removed copper zone on F.Cu, net V_SERVO_E0
Other:
- board size 88.1 x 95.6 mm -> 68.3 x 95.1 mm
- board text added: "PA0"
- board text added: "PA1"
- board text added: "PA2"
- board text added: "PA3"
- board text added: "PA6"
- board text added: "PA7"
- board text added: "PB0"
- board text added: "PB1"
- board text added: "PB10"
- board text added: "PB3"
- board text added: "PB6"
- board text added: "PB7"
- board text added: "RX"
- board text added: "TX"
- board text added: "VCC"
- board text added: "VSR"
- board text added: "VST 5.5V-24V"
- board text removed: "-"
- board text removed: "2"
- board text removed: "3"
- board text removed: "5V"
- board text removed: "A0 A3 A2"
- board text removed: "A0 A3 A2 A1 B6 B7"
- board text removed: "A1 B6 B7"
- board text removed: "A6 A7 B0 B1 B10 B3"
- board text removed: "A6 A7 B8 B1"
- board text removed: "B10"
- board text removed: "B3"
- board text removed: "EB0"
- board text removed: "EB1"
- board text removed: "EB2"
- board text removed: "EB3"
- board text removed: "EXP0"
- board text removed: "EXP1"
- board text removed: "I2C"
- board text removed: "P0"
- board text removed: "P0 P1 P2 P3 P4 P5"
- board text removed: "P1"
- board text removed: "P2"
- board text removed: "P3"
- board text removed: "P4"
- board text removed: "P5"
- board text removed: "P5 P4 P3 P2 P1 P0"
- board text removed: "RXD"
- board text removed: "S2"
- board text removed: "S3"
- board text removed: "S4"
- board text removed: "S5"
- board text removed: "SCL"
- board text removed: "SDA"
- board text removed: "SERVO"
- board text removed: "STEPPER 5.5V"
- board text removed: "TXD"
- board text removed: "UART"
- board text removed: "Vsrv"
- board text removed: "to 24V"

Commit message: working
Parts:
- removed the REF** at (176.6, 166.0)
- removed the REF** at (144.7, 119.3)
- removed the REF** at (144.7, 109.6)
- removed the REF** at (144.7, 99.8)
- removed the REF** at (144.7, 90.0)
- added C120: 100nF 16V, Capacitor_SMD:C_0402_1005Metric, F.Cu at (126.2, 114.0)
- added C2: 100nF 16V, Capacitor_SMD:C_0402_1005Metric, F.Cu at (131.5, 114.0)
- added C4: 100nF 16V, Capacitor_SMD:C_0402_1005Metric, F.Cu at (120.9, 114.0)
- added J12: HSES, Connector_PinHeader_1.00mm:PinHeader_1x03_P1.00mm_Vertical, F.Cu at (126.2, 115.0)
- added J5: HSES, Connector_PinHeader_1.00mm:PinHeader_1x03_P1.00mm_Vertical, B.Cu at (132.4, 116.4)
- added J8: HSES, Connector_PinHeader_1.00mm:PinHeader_1x03_P1.00mm_Vertical, F.Cu at (120.9, 115.3)
- added REF**: ToolingHole, MountingHole:MountingHole_3.2mm_M3, F.Cu at (180.0, 142.0)
- added U13: CH912LSR, Package_TO_SOT_SMD:SOT-23W, F.Cu at (120.9, 116.5)
- added U14: CH912LSR, Package_TO_SOT_SMD:SOT-23W, F.Cu at (126.2, 116.5)
- added U2: CH912LSR, Package_TO_SOT_SMD:SOT-23W, F.Cu at (131.5, 116.5)
- U3: value STM32F411RCT6 -> STM32F411RET6
Routing:
- net Net-(C120-Pad1): track 0.00 -> 5.99 mm
- net Net-(C4-Pad1): track 0.00 -> 5.99 mm
- net Net-(C2-Pad1): track 0.00 -> 5.99 mm
- net Net-(C4-Pad2): track 0.00 -> 3.17 mm
- net Net-(C120-Pad2): track 0.00 -> 3.17 mm
- net Net-(C2-Pad2): track 0.00 -> 3.17 mm
- net Net-(J12-Pad1): track 0.00 -> 0.99 mm
- net Net-(J8-Pad1): track 0.00 -> 0.99 mm
- net Net-(J5-Pad1): track 0.00 -> 0.99 mm
- removed copper zone on B.Cu, net (none)
- removed copper zone on In1.Cu, net (none)
- removed copper zone on In2.Cu, net (none)
Other:
- outline, holes or cut-outs redrawn
- board text added: "-"
- board text added: "s"

Commit message: going to rearrange everything
Parts:
- added C1: 1.0uF 25V, Capacitor_SMD:C_0402_1005Metric, F.Cu at (20.9, 145.9)
- added C10: 4.7uF 10V, Capacitor_SMD:C_0402_1005Metric, F.Cu at (-1.93, 134.1)
- added C100: 470pF 50V, Capacitor_SMD:C_0402_1005Metric, F.Cu at (-26.4, 176.5)
- added C101: 470pF 50V, Capacitor_SMD:C_0402_1005Metric, F.Cu at (-19.0, 174.6)
- added C102: 470pF 50V, Capacitor_SMD:C_0402_1005Metric, F.Cu at (14.2, 173.2)
- added C103: 470pF 50V, Capacitor_SMD:C_0402_1005Metric, F.Cu at (20.6, 172.6)
- added C104: 470pF 50V, Capacitor_SMD:C_0402_1005Metric, F.Cu at (-6.04, 174.5)
- added C105: 470pF 50V, Capacitor_SMD:C_0402_1005Metric, F.Cu at (-0.88, 174.0)
- added C106: 470pF 50V, Capacitor_SMD:C_0402_1005Metric, F.Cu at (-23.3, 173.6)
- added C107: 470pF 50V, Capacitor_SMD:C_0402_1005Metric, F.Cu at (-22.1, 174.7)
- added C108: 33nF 50V, Capacitor_SMD:C_0402_1005Metric, F.Cu at (-10.7, 166.0)
- added C109: 33nF 50V, Capacitor_SMD:C_0402_1005Metric, F.Cu at (12.2, 166.1)
- added C11: 4.7uF 10V, Capacitor_SMD:C_0402_1005Metric, F.Cu at (16.4, 136.2)
- added C110: 33nF 50V, Capacitor_SMD:C_0402_1005Metric, F.Cu at (28.9, 165.1)
- added C111: 33nF 50V, Capacitor_SMD:C_0402_1005Metric, F.Cu at (4.00, 165.1)
- added C112: 33nF 50V, Capacitor_SMD:C_0402_1005Metric, F.Cu at (0.89, 166.1)
- added C113: 33nF 50V, Capacitor_SMD:C_0402_1005Metric, F.Cu at (20.0, 164.5)
- added C114: 33nF 50V, Capacitor_SMD:C_0402_1005Metric, F.Cu at (28.9, 166.1)
- added C115: 33nF 50V, Capacitor_SMD:C_0402_1005Metric, F.Cu at (23.8, 165.1)
- added C116: 33nF 50V, Capacitor_SMD:C_0402_1005Metric, F.Cu at (-4.83, 164.5)
- added C117: 33nF 50V, Capacitor_SMD:C_0402_1005Metric, F.Cu at (-6.76, 164.5)
- added C118: 33nF 50V, Capacitor_SMD:C_0402_1005Metric, F.Cu at (19.0, 164.5)
- added C119: 33nF 50V, Capacitor_SMD:C_0402_1005Metric, F.Cu at (23.8, 166.1)
- added C12: 1.0uF 25V, Capacitor_SMD:C_0402_1005Metric, F.Cu at (15.9, 138.0)
- added C13: 100nF 16V, Capacitor_SMD:C_0402_1005Metric, F.Cu at (4.16, 157.3)
- added C14: 100nF 16V, Capacitor_SMD:C_0402_1005Metric, F.Cu at (3.28, 130.3)
- added C15: 100nF 16V, Capacitor_SMD:C_0402_1005Metric, F.Cu at (12.2, 157.3)
- added C16: 100nF 16V, Capacitor_SMD:C_0402_1005Metric, F.Cu at (14.8, 138.4)
- added C17: 100nF 16V, Capacitor_SMD:C_0402_1005Metric, F.Cu at (10.7, 131.0)
- added C18: 100nF 16V, Capacitor_SMD:C_0402_1005Metric, F.Cu at (-15.3, 157.1)
- added C19: 470pF 50V, Capacitor_SMD:C_0402_1005Metric, F.Cu at (25.5, 175.3)
- added C20: 470pF 50V, Capacitor_SMD:C_0402_1005Metric, F.Cu at (12.5, 176.4)
- added C21: 470pF 50V, Capacitor_SMD:C_0402_1005Metric, F.Cu at (5.54, 175.2)
- added C22: 470pF 50V, Capacitor_SMD:C_0402_1005Metric, F.Cu at (-0.74, 144.7)
- added C23: 470pF 50V, Capacitor_SMD:C_0402_1005Metric, F.Cu at (-14.3, 175.3)
- added C24: 470pF 50V, Capacitor_SMD:C_0402_1005Metric, F.Cu at (-25.9, 158.8)
- added C3: 1.0uF 25V, Capacitor_SMD:C_0402_1005Metric, F.Cu at (15.2, 144.7)
- added C31: 100nF 16V, Capacitor_SMD:C_0402_1005Metric, F.Cu at (28.4, 173.5)
- added C32: 100nF 16V, Capacitor_SMD:C_0402_1005Metric, F.Cu at (30.0, 159.3)
- added C33: 100nF 16V, Capacitor_SMD:C_0402_1005Metric, F.Cu at (8.55, 173.4)
- added C34: 100nF 16V, Capacitor_SMD:C_0402_1005Metric, F.Cu at (10.4, 158.0)
- added C35: 100nF 16V, Capacitor_SMD:C_0402_1005Metric, F.Cu at (-11.2, 173.4)
- added C36: 100nF 16V, Capacitor_SMD:C_0402_1005Metric, F.Cu at (-11.0, 157.3)
- added C37: 100nF 16V, Capacitor_SMD:C_0402_1005Metric, F.Cu at (24.4, 173.5)
- added C38: 100nF 16V, Capacitor_SMD:C_0402_1005Metric, F.Cu at (4.54, 173.4)
- added C39: 100nF 16V, Capacitor_SMD:C_0402_1005Metric, F.Cu at (-15.2, 173.4)
- added C40: 100nF 16V, Capacitor_SMD:C_0402_1005Metric, F.Cu at (24.2, 157.3)
- added C41: 100nF 16V, Capacitor_SMD:C_0402_1005Metric, F.Cu at (-1.21, 134.8)
- added C42: 100nF 16V, Capacitor_SMD:C_0402_1005Metric, F.Cu at (-3.45, 157.3)
- added C43: 33nF 50V, Capacitor_SMD:C_0402_1005Metric, F.Cu at (-24.6, 164.1)
- added C44: 33nF 50V, Capacitor_SMD:C_0402_1005Metric, F.Cu at (-18.9, 166.1)
- added C45: 33nF 50V, Capacitor_SMD:C_0402_1005Metric, F.Cu at (-26.0, 164.6)
- added C46: 33nF 50V, Capacitor_SMD:C_0402_1005Metric, F.Cu at (-5.79, 164.5)
- added C47: 33nF 50V, Capacitor_SMD:C_0402_1005Metric, F.Cu at (-26.0, 162.8)
- added C48: 33nF 50V, Capacitor_SMD:C_0402_1005Metric, F.Cu at (-15.8, 165.1)
- added C49: 22nF 50V, Capacitor_SMD:C_0402_1005Metric, F.Cu at (30.0, 161.2)
- added C5: 15pF, Capacitor_SMD:C_0402_1005Metric, F.Cu at (13.0, 132.6)
- added C50: 22nF 50V, Capacitor_SMD:C_0402_1005Metric, F.Cu at (10.2, 161.3)
- added C51: 22nF 50V, Capacitor_SMD:C_0402_1005Metric, F.Cu at (-9.05, 162.1)
- added C53: 4.7uF 10V, Capacitor_SMD:C_0402_1005Metric, F.Cu at (26.6, 157.8)
- added C54: 4.7uF 10V, Capacitor_SMD:C_0402_1005Metric, F.Cu at (6.83, 157.8)
- added C55: 4.7uF 10V, Capacitor_SMD:C_0402_1005Metric, F.Cu at (-13.0, 157.8)
- added C56: 470pF 50V, Capacitor_SMD:C_0402_1005Metric, F.Cu at (23.4, 173.5)
- added C57: 470pF 50V, Capacitor_SMD:C_0402_1005Metric, F.Cu at (29.4, 173.5)
- added C58: 470pF 50V, Capacitor_SMD:C_0402_1005Metric, F.Cu at (3.56, 173.4)
- added C59: 470pF 50V, Capacitor_SMD:C_0402_1005Metric, F.Cu at (9.54, 173.4)
- added C6: 15pF, Capacitor_SMD:C_0402_1005Metric, F.Cu at (13.1, 130.7)
- added C60: 470pF 50V, Capacitor_SMD:C_0402_1005Metric, F.Cu at (-16.2, 173.4)
- added C61: 470pF 50V, Capacitor_SMD:C_0402_1005Metric, F.Cu at (-10.2, 173.4)
- added C62: 470pF 50V, Capacitor_SMD:C_0402_1005Metric, F.Cu at (25.4, 173.5)
- added C63: 470pF 50V, Capacitor_SMD:C_0402_1005Metric, F.Cu at (27.4, 173.5)
- added C64: 470pF 50V, Capacitor_SMD:C_0402_1005Metric, F.Cu at (5.54, 173.4)
- added C65: 470pF 50V, Capacitor_SMD:C_0402_1005Metric, F.Cu at (7.54, 173.4)
- added C66: 470pF 50V, Capacitor_SMD:C_0402_1005Metric, F.Cu at (-14.2, 173.4)
- added C67: 470pF 50V, Capacitor_SMD:C_0402_1005Metric, F.Cu at (-12.3, 173.4)
- added C7: 15pF, Capacitor_SMD:C_0402_1005Metric, F.Cu at (20.2, 134.3)
- added C72: 100nF 16V, Capacitor_SMD:C_0402_1005Metric, F.Cu at (17.6, 166.6)
- added C73: 100nF 16V, Capacitor_SMD:C_0402_1005Metric, F.Cu at (16.6, 157.3)
- added C74: 100nF 16V, Capacitor_SMD:C_0402_1005Metric, F.Cu at (-1.65, 168.4)
- added C75: 100nF 16V, Capacitor_SMD:C_0402_1005Metric, F.Cu at (1.81, 157.3)
- added C76: 100nF 16V, Capacitor_SMD:C_0402_1005Metric, F.Cu at (-19.4, 167.8)
- added C77: 100nF 16V, Capacitor_SMD:C_0402_1005Metric, F.Cu at (-18.4, 157.8)
- added C78: 100nF 16V, Capacitor_SMD:C_0402_1005Metric, F.Cu at (14.8, 168.4)
- added C79: 100nF 16V, Capacitor_SMD:C_0402_1005Metric, F.Cu at (-4.33, 167.3)
- added C8: 15pF, Capacitor_SMD:C_0402_1005Metric, F.Cu at (20.2, 132.2)
- added C80: 100nF 16V, Capacitor_SMD:C_0402_1005Metric, F.Cu at (-24.6, 165.5)
- added C81: 100nF 16V, Capacitor_SMD:C_0402_1005Metric, F.Cu at (14.8, 136.2)
- added C82: 100nF 16V, Capacitor_SMD:C_0402_1005Metric, F.Cu at (-23.3, 157.3)
- added C83: 100nF 16V, Capacitor_SMD:C_0402_1005Metric, F.Cu at (4.24, 145.1)
- added C84: 33nF 50V, Capacitor_SMD:C_0402_1005Metric, F.Cu at (9.11, 166.0)
- added C85: 33nF 50V, Capacitor_SMD:C_0402_1005Metric, F.Cu at (-10.7, 165.1)
- added C86: 33nF 50V, Capacitor_SMD:C_0402_1005Metric, F.Cu at (-15.8, 166.0)
- added C87: 33nF 50V, Capacitor_SMD:C_0402_1005Metric, F.Cu at (18.0, 164.5)
- added C88: 33nF 50V, Capacitor_SMD:C_0402_1005Metric, F.Cu at (9.11, 165.1)
- added C89: 33nF 50V, Capacitor_SMD:C_0402_1005Metric, F.Cu at (4.00, 166.0)
- added C9: 100nF 16V, Capacitor_SMD:C_0402_1005Metric, F.Cu at (24.1, 135.3)
- added C90: 22nF 50V, Capacitor_SMD:C_0402_1005Metric, F.Cu at (18.9, 161.8)
- added C91: 22nF 50V, Capacitor_SMD:C_0402_1005Metric, F.Cu at (2.40, 161.3)
- added C92: 22nF 50V, Capacitor_SMD:C_0402_1005Metric, F.Cu at (-17.4, 161.2)
- added C93: 4.7uF 10V, Capacitor_SMD:C_0402_1005Metric, F.Cu at (14.6, 157.8)
- added C94: 4.7uF 10V, Capacitor_SMD:C_0402_1005Metric, F.Cu at (-0.97, 157.8)
- added C95: 4.7uF 10V, Capacitor_SMD:C_0402_1005Metric, F.Cu at (-20.8, 157.8)
- added C96: 470pF 50V, Capacitor_SMD:C_0402_1005Metric, F.Cu at (13.1, 171.7)
- added C97: 470pF 50V, Capacitor_SMD:C_0402_1005Metric, F.Cu at (20.6, 170.5)
- added C98: 470pF 50V, Capacitor_SMD:C_0402_1005Metric, F.Cu at (-6.72, 175.2)
- added C99: 470pF 50V, Capacitor_SMD:C_0402_1005Metric, F.Cu at (0.56, 174.0)
- added D1: B5819W, Diode_SMD:D_SOD-123, F.Cu at (22.3, 143.9)
- added D2: Blue, LED_SMD:LED_0603_1608Metric, F.Cu at (-3.73, 134.4)
- added D3: B5819W, Diode_SMD:D_SOD-123, F.Cu at (30.2, 154.8)
- added J1: USB_C-SIGNAL, Connector_USB:USB_C_Receptacle_HRO_TYPE-C-31-M-12, F.Cu at (-31.6, 148.6)
- added J16: ADC0, Connector_JST:JST_PH_B2B-PH-K_1x02_P2.00mm_Vertical, F.Cu at (30.4, 157.7)
- added J16: ADC0, Connector_JST:JST_PH_B2B-PH-K_1x02_P2.00mm_Vertical, F.Cu at (35.2, 157.7)
- added J16: ADC0, Connector_JST:JST_PH_B2B-PH-K_1x02_P2.00mm_Vertical, F.Cu at (35.7, 137.7)
- added J16: ADC0, Connector_JST:JST_PH_B2B-PH-K_1x02_P2.00mm_Vertical, F.Cu at (30.9, 137.7)
- added J17: ESTP0, Connector_JST:JST_PH_B3B-PH-K_1x03_P2.00mm_Vertical, F.Cu at (-21.4, 139.3)
- added J18: ESTP1, Connector_JST:JST_PH_B3B-PH-K_1x03_P2.00mm_Vertical, F.Cu at (10.5, 158.3)
- added J19: ESTP2, Connector_JST:JST_PH_B3B-PH-K_1x03_P2.00mm_Vertical, F.Cu at (-3.38, 139.3)
- added J20: ESTP3, Connector_JST:JST_PH_B3B-PH-K_1x03_P2.00mm_Vertical, F.Cu at (-7.46, 158.3)
- added J21: ESTP4, Connector_JST:JST_PH_B3B-PH-K_1x03_P2.00mm_Vertical, F.Cu at (14.6, 139.3)
- added J22: ESTP5, Connector_JST:JST_PH_B3B-PH-K_1x03_P2.00mm_Vertical, F.Cu at (-25.5, 158.3)
- added J23: POWER, Connector_AMASS:AMASS_MR30PW-M_1x03_P3.50mm_Horizontal, F.Cu at (12.8, 145.2)
- added J25: SERV0, Connector_JST:JST_PH_B3B-PH-K_1x03_P2.00mm_Vertical, F.Cu at (-29.4, 157.1)
- added J25: SERV0, Connector_JST:JST_PH_B3B-PH-K_1x03_P2.00mm_Vertical, F.Cu at (-29.4, 136.9)
- added J26: SERV1, Connector_JST:JST_PH_B3B-PH-K_1x03_P2.00mm_Vertical, F.Cu at (-33.4, 160.5)
- added J26: SERV1, Connector_JST:JST_PH_B3B-PH-K_1x03_P2.00mm_Vertical, F.Cu at (-33.4, 140.3)
- added J6: PWM0_OUT, Connector_AMASS:AMASS_XT30U-F_1x02_P5.0mm_Vertical, F.Cu at (45.6, 138.6)
- added J7: PWM1_OUT, Connector_AMASS:AMASS_XT30U-F_1x02_P5.0mm_Vertical, F.Cu at (45.1, 158.8)
- added P1: STP0, Connector_JST:JST_PH_B4B-PH-K_1x04_P2.00mm_Vertical, F.Cu at (18.5, 158.3)
- added P2: STP2, Connector_JST:JST_PH_B4B-PH-K_1x04_P2.00mm_Vertical, F.Cu at (6.53, 157.3)
- added P3: STP4, Connector_JST:JST_PH_B4B-PH-K_1x04_P2.00mm_Vertical, F.Cu at (-11.5, 157.3)
- added P4: STP1, Connector_JST:JST_PH_B4B-PH-K_1x04_P2.00mm_Vertical, F.Cu at (-11.4, 139.3)
- added P5: STP3, Connector_JST:JST_PH_B4B-PH-K_1x04_P2.00mm_Vertical, F.Cu at (6.62, 139.3)
- added P6: STP5, Connector_JST:JST_PH_B4B-PH-K_1x04_P2.00mm_Vertical, F.Cu at (24.6, 139.3)
- added P9: UART, Connector_JST:JST_PH_B4B-PH-K_1x04_P2.00mm_Vertical, F.Cu at (26.3, 190.8)
- added R100: 330R, Resistor_SMD:R_0402_1005Metric, F.Cu at (-2.25, 145.1)
- added R101: 330R, Resistor_SMD:R_0402_1005Metric, F.Cu at (-15.8, 175.8)
- added R102: 330R, Resistor_SMD:R_0402_1005Metric, F.Cu at (-26.9, 158.8)
- added R103: 330R, Resistor_SMD:R_0402_1005Metric, F.Cu at (33.2, 166.6)
- added R104: 330R, Resistor_SMD:R_0402_1005Metric, F.Cu at (34.3, 166.6)
- added R17: 33k, Resistor_SMD:R_0402_1005Metric, F.Cu at (-4.39, 142.5)
- added R29: 5.1k, Resistor_SMD:R_0402_1005Metric, F.Cu at (-1.24, 136.8)
- added R3: 5.1k, Resistor_SMD:R_0402_1005Metric, F.Cu at (30.3, 151.4)
- added R30: 33k, Resistor_SMD:R_0402_1005Metric, F.Cu at (-3.42, 132.2)
- added R32: 330R, Resistor_SMD:R_0402_1005Metric, F.Cu at (-9.02, 130.5)
- added R33: 330R, Resistor_SMD:R_0402_1005Metric, F.Cu at (-6.54, 130.5)
- added R34: 330R, Resistor_SMD:R_0402_1005Metric, F.Cu at (-6.54, 131.5)
- added R35: 330R, Resistor_SMD:R_0402_1005Metric, F.Cu at (-6.54, 132.5)
- added R36: 330R, Resistor_SMD:R_0402_1005Metric, F.Cu at (-6.54, 133.5)
- added R37: 330R, Resistor_SMD:R_0402_1005Metric, F.Cu at (-6.54, 134.5)
- added R38: 330R, Resistor_SMD:R_0402_1005Metric, F.Cu at (-9.02, 129.5)
- added R4: 5.1k, Resistor_SMD:R_0402_1005Metric, F.Cu at (30.3, 149.0)
- added R40: 330R, Resistor_SMD:R_0402_1005Metric, F.Cu at (7.36, 129.3)
- added R41: 330R, Resistor_SMD:R_0402_1005Metric, F.Cu at (10.0, 129.3)
- added R42: 330R, Resistor_SMD:R_0402_1005Metric, F.Cu at (-10.6, 132.2)
- added R43: 330R, Resistor_SMD:R_0402_1005Metric, F.Cu at (13.1, 142.9)
- added R44: 330R, Resistor_SMD:R_0402_1005Metric, F.Cu at (13.8, 142.2)
- added R45: 10k, Resistor_SMD:R_0402_1005Metric, F.Cu at (22.9, 142.1)
- added R47: 1R, Resistor_SMD:R_0402_1005Metric, F.Cu at (24.7, 168.1)
- added R48: 1R, Resistor_SMD:R_0402_1005Metric, F.Cu at (24.7, 167.1)
- added R49: 1R, Resistor_SMD:R_0402_1005Metric, F.Cu at (24.7, 170.0)
- added R50: 1R, Resistor_SMD:R_0402_1005Metric, F.Cu at (24.7, 169.0)
- added R51: 1R, Resistor_SMD:R_0402_1005Metric, F.Cu at (17.3, 142.0)
- added R51: 1R, Resistor_SMD:R_0402_1005Metric, F.Cu at (21.3, 142.0)
- added R51: 1R, Resistor_SMD:R_0402_1005Metric, F.Cu at (17.3, 155.4)
- added R51: 1R, Resistor_SMD:R_0402_1005Metric, F.Cu at (21.3, 155.5)
- added R52: 1R, Resistor_SMD:R_0402_1005Metric, F.Cu at (20.3, 142.0)
- added R52: 1R, Resistor_SMD:R_0402_1005Metric, F.Cu at (26.2, 142.0)
- added R52: 1R, Resistor_SMD:R_0402_1005Metric, F.Cu at (20.3, 155.4)
- added R52: 1R, Resistor_SMD:R_0402_1005Metric, F.Cu at (26.2, 155.5)
- added R53: 1R, Resistor_SMD:R_0402_1005Metric, F.Cu at (19.3, 142.0)
- added R53: 1R, Resistor_SMD:R_0402_1005Metric, F.Cu at (25.2, 142.0)
- added R53: 1R, Resistor_SMD:R_0402_1005Metric, F.Cu at (19.3, 155.4)
- added R53: 1R, Resistor_SMD:R_0402_1005Metric, F.Cu at (25.2, 155.5)
- added R54: 1R, Resistor_SMD:R_0402_1005Metric, F.Cu at (24.2, 142.0)
- added R54: 1R, Resistor_SMD:R_0402_1005Metric, F.Cu at (18.3, 142.0)
- added R54: 1R, Resistor_SMD:R_0402_1005Metric, F.Cu at (18.3, 155.4)
- added R54: 1R, Resistor_SMD:R_0402_1005Metric, F.Cu at (24.2, 155.5)
- added R55: 1R, Resistor_SMD:R_0402_1005Metric, F.Cu at (4.89, 168.0)
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Other:
- board size 68.3 x 95.1 mm -> 213 x 95.1 mm

Commit message: partial
Parts:
- removed the C1 at (20.9, 145.9)
- removed the C10 at (-1.93, 134.1)
- removed C100 (x2), C101 (x2), C102 (x2), C103 (x2), C104 (x2), C105 (x2), C106 (x2), C107 (x2), C56 (x2), C57 (x2), C58 (x2), C59 (x2), C60 (x2), C61 (x2), C62 (x2), C63 (x2), C64 (x2), C65 (x2), C66 (x2), C67 (x2), C96 (x2), C97 (x2), C98 (x2), C99 (x2): 470pF 50V, Capacitor_SMD:C_0402_1005Metric
- removed the C108 at (-10.7, 166.0)
- removed the C108 at (133.9, 157.4)
- removed C109 (x2), C110 (x2), C111 (x2), C115 (x2), C116 (x2), C117 (x2), C43 (x2), C44 (x2), C45 (x2), C84 (x2), C85 (x2), C86 (x2): 33nF 50V, Capacitor_SMD:C_0402_1005Metric
- removed the C11 at (16.4, 136.2)
- removed the C112 at (0.89, 166.1)
- removed the C112 at (145.5, 157.4)
- removed the C113 at (20.0, 164.5)
- removed the C113 at (164.6, 155.8)
- removed the C114 at (28.9, 166.1)
- removed the C114 at (173.6, 157.4)
- removed the C118 at (19.0, 164.5)
- removed the C118 at (163.6, 155.8)
- removed the C119 at (23.8, 166.1)
- removed the C119 at (168.4, 157.4)
- removed the C12 at (15.9, 138.0)
- removed the C13 at (4.16, 157.3)
- removed the C14 at (3.28, 130.3)
- removed the C15 at (12.2, 157.3)
- removed the C16 at (14.8, 138.4)
- removed the C17 at (10.7, 131.0)
- removed the C18 at (-15.3, 157.1)
- removed the C19 at (25.5, 175.3)
- removed the C20 at (12.5, 176.4)
- removed the C21 at (5.54, 175.2)
- removed the C22 at (-0.74, 144.7)
- removed the C23 at (-14.3, 175.3)
- removed the C24 at (-25.9, 158.8)
- removed the C3 at (15.2, 144.7)
- removed C31 (x2), C33 (x2), C35 (x2), C37 (x2), C38 (x2), C39 (x2), C72 (x2), C74 (x2), C76 (x2), C78 (x2), C79 (x2), C80 (x2): 100nF 16V, Capacitor_SMD:C_0402_1005Metric
- removed the C32 at (30.0, 159.3)
- removed the C34 at (10.4, 158.0)
- removed the C36 at (-11.0, 157.3)
- removed the C40 at (24.2, 157.3)
- removed the C41 at (-1.21, 134.8)
- removed the C42 at (-3.45, 157.3)
- removed the C46 at (-5.79, 164.5)
- removed the C46 at (138.8, 155.8)
- removed the C47 at (-26.0, 162.8)
- removed the C47 at (118.7, 154.1)
- removed the C48 at (-15.8, 165.1)
- removed the C48 at (128.9, 156.4)
- removed the C49 at (30.0, 161.2)
- removed the C5 at (13.0, 132.6)
- removed the C50 at (10.2, 161.3)
- removed the C51 at (-9.05, 162.1)
- removed the C53 at (26.6, 157.8)
- removed the C54 at (6.83, 157.8)
- removed the C55 at (-13.0, 157.8)
- removed the C6 at (13.1, 130.7)
- removed the C7 at (20.2, 134.3)
- removed the C73 at (16.6, 157.3)
- removed the C75 at (1.81, 157.3)
- removed the C77 at (-18.4, 157.8)
- removed the C8 at (20.2, 132.2)
- removed the C81 at (14.8, 136.2)
- removed the C82 at (-23.3, 157.3)
- removed the C83 at (4.24, 145.1)
- removed the C87 at (18.0, 164.5)
- removed the C87 at (162.7, 155.8)
- removed the C88 at (9.11, 165.1)
- removed the C88 at (153.7, 156.4)
- removed the C89 at (4.00, 166.0)
- removed the C89 at (148.6, 157.4)
- removed the C9 at (24.1, 135.3)
- removed the C90 at (18.9, 161.8)
- removed the C91 at (2.40, 161.3)
- removed the C92 at (-17.4, 161.2)
- removed the C93 at (14.6, 157.8)
- removed the C94 at (-0.97, 157.8)
- removed the C95 at (-20.8, 157.8)
- removed the D1 at (22.3, 143.9)
- removed the D2 at (-3.73, 134.4)
- removed the D3 at (30.2, 154.8)
- removed the J1 at (-31.6, 148.6)
- removed the J16 at (30.4, 157.7)
- removed the J16 at (35.2, 157.7)
- removed the J16 at (35.7, 137.7)
- removed the J16 at (30.9, 137.7)
- removed the J17 at (-21.4, 139.3)
- removed the J18 at (10.5, 158.3)
- removed the J19 at (-3.38, 139.3)
- removed the J20 at (-7.46, 158.3)
- removed the J21 at (14.6, 139.3)
- removed the J22 at (-25.5, 158.3)
- removed the J23 at (12.8, 145.2)
- removed the J23 at (172.0, 124.7)
- removed the J25 at (-29.4, 157.1)
- removed the J25 at (-29.4, 136.9)
- removed the J26 at (-33.4, 160.5)
- removed the J26 at (-33.4, 140.3)
- removed the J6 at (45.6, 138.6)
- removed the J7 at (45.1, 158.8)
- removed the P1 at (18.5, 158.3)
- removed the P2 at (6.53, 157.3)
- removed the P3 at (-11.5, 157.3)
- removed the P4 at (-11.4, 139.3)
- removed the P5 at (6.62, 139.3)
- removed the P6 at (24.6, 139.3)
- removed the P9 at (26.3, 190.8)
- removed the R100 at (-2.25, 145.1)
- removed the R101 at (-15.8, 175.8)
- removed the R102 at (-26.9, 158.8)
- removed the R103 at (33.2, 166.6)
- removed the R103 at (177.8, 157.9)
- removed the R104 at (34.3, 166.6)
- removed the R104 at (178.9, 157.9)
- removed the R17 at (-4.39, 142.5)
- removed the R29 at (-1.24, 136.8)
- removed the R3 at (30.3, 151.4)
- removed the R30 at (-3.42, 132.2)
- removed the R32 at (-9.02, 130.5)
- removed the R33 at (-6.54, 130.5)
- removed the R34 at (-6.54, 131.5)
- removed the R35 at (-6.54, 132.5)
- removed the R36 at (-6.54, 133.5)
- removed the R37 at (-6.54, 134.5)
- removed the R38 at (-9.02, 129.5)
- removed the R4 at (30.3, 149.0)
- removed the R40 at (7.36, 129.3)
- removed the R41 at (10.0, 129.3)
- removed the R42 at (-10.6, 132.2)
- removed the R43 at (13.1, 142.9)
- removed the R44 at (13.8, 142.2)
- removed the R45 at (22.9, 142.1)
- removed the R47 at (24.7, 168.1)
- removed the R47 at (169.3, 159.4)
- removed R48 (x2), R49 (x2), R50 (x2), R51 (x5), R52 (x5), R53 (x5), R54 (x5), R55 (x2), R56 (x2), R57 (x2), R58 (x2), R59 (x2), R60 (x2), R61 (x2), R62 (x2), R63 (x2), R64 (x2), R65 (x2), R66 (x2), R67 (x2), R68 (x2), R69 (x2), R70 (x2), R73 (x2), R74 (x2), R75 (x2), R76 (x2), R77 (x2), R78 (x2), R79 (x2), R80 (x2), R81 (x2), R82 (x2), R83 (x2), R84 (x2), R85 (x2), R86 (x2), R87 (x2), R88 (x2), R89 (x2), R90 (x2), R91 (x2), R92 (x2), R93 (x2), R94 (x2), R95 (x2), R96 (x2): 1R, Resistor_SMD:R_0402_1005Metric
- removed the R7 at (32.0, 160.9)
- removed the R7 at (176.7, 152.3)
- removed the R8 at (32.0, 159.7)
- removed the R8 at (176.7, 151.1)
- removed the R97 at (24.0, 175.8)
- removed the R98 at (11.5, 176.4)
- removed the R99 at (4.05, 175.6)
- removed the REF** at (-11.8, 160.4)
- removed the REF** at (-22.8, 132.6)
- removed the REF** at (-4.71, 164.9)
- removed the REF** at (-22.7, 165.0)
- removed the REF** at (12.9, 164.7)
- removed the REF** at (20.4, 138.7)
- removed the REF** at (35.4, 150.7)
- removed the REF** at (20.4, 158.7)
- removed the REF** at (-7.24, 158.7)
- removed the REF** at (-7.24, 138.7)
- removed the REF** at (-16.4, 160.4)
- removed the REF** at (175.4, 78.8)
- removed the REF** at (155.4, 78.8)
- removed the REF** at (165.0, 130.0)
- removed the REF** at (137.4, 130.0)
- removed the REF** at (165.0, 150.0)
- removed the REF** at (137.4, 150.0)
- removed the REF** at (155.4, 115.2)
- removed the REF** at (37.4, 173.8)
- removed the REF** at (-31.6, 167.1)
- removed the REF** at (-31.6, 164.6)
- removed the REF** at (-31.7, 129.9)
- removed the REF** at (-31.7, 132.4)
- removed the REF** at (12.7, 132.3)
- removed the REF** at (-4.86, 132.5)
- removed the SW1 at (23.3, 131.9)
- removed the SW2 at (-7.78, 143.8)
- removed the TP1 at (-2.80, 137.3)
- removed the TP2 at (-2.80, 139.9)
- removed the TP3 at (-2.80, 142.4)
- removed the U1 at (17.8, 143.9)
- removed the U10 at (22.3, 132.2)
- removed the U11 at (4.08, 132.3)
- removed the U12 at (-14.1, 165.5)
- removed the U3 at (-5.38, 148.7)
- removed the U5 at (3.90, 164.8)
- removed the U6 at (21.1, 165.5)
- removed the U7 at (-13.3, 132.5)
- removed the Y1 at (15.3, 131.4)
- removed the Y2 at (18.4, 133.3)
- added C108: 100nF 50V, Capacitor_SMD:C_0603_1608Metric, F.Cu at (29.7, -10.9)
- added C112: 100nF 50V, Capacitor_SMD:C_0603_1608Metric, F.Cu at (11.7, -10.9)
- added C113: 100nF 50V, Capacitor_SMD:C_0603_1608Metric, F.Cu at (15.3, -10.9)
- added C114: 100nF 50V, Capacitor_SMD:C_0603_1608Metric, F.Cu at (56.3, -10.9)
- added C118: 100nF 50V, Capacitor_SMD:C_0603_1608Metric, F.Cu at (33.3, -10.9)
- added C119: 100nF 50V, Capacitor_SMD:C_0603_1608Metric, F.Cu at (11.7, 10.9)
- added C46: 100nF 50V, Capacitor_SMD:C_0603_1608Metric, F.Cu at (33.3, 10.9)
- added C47: 100nF 50V, Capacitor_SMD:C_0603_1608Metric, F.Cu at (52.7, 10.9)
- added C48: 100nF 50V, Capacitor_SMD:C_0603_1608Metric, F.Cu at (52.7, -10.9)
- added C87: 100nF 50V, Capacitor_SMD:C_0603_1608Metric, F.Cu at (56.3, 10.9)
- added C88: 100nF 50V, Capacitor_SMD:C_0603_1608Metric, F.Cu at (29.7, 10.9)
- added C89: 100nF 50V, Capacitor_SMD:C_0603_1608Metric, F.Cu at (15.3, 10.9)
- added J23: POWER, Connector_AMASS:AMASS_MR30PW-M_1x03_P3.50mm_Horizontal, F.Cu at (56.0, -3.50)
- added R103: 330R, Resistor_SMD:R_0402_1005Metric, F.Cu at (28.1, 43.0)
- added R104: 330R, Resistor_SMD:R_0402_1005Metric, F.Cu at (32.5, 40.5)
- added R13: R25, Resistor_SMD:R_0805_2012Metric, F.Cu at (15.5, -12.6)
- added R14: R25, Resistor_SMD:R_0805_2012Metric, F.Cu at (52.5, -12.6)
- added R15: R25, Resistor_SMD:R_0805_2012Metric, F.Cu at (56.5, -12.6)
- added R16: R25, Resistor_SMD:R_0805_2012Metric, F.Cu at (33.5, 12.6)
- added R18: R25, Resistor_SMD:R_0805_2012Metric, F.Cu at (29.5, 12.6)
- added R19: R25, Resistor_SMD:R_0805_2012Metric, F.Cu at (29.5, -12.6)
- added R20: R25, Resistor_SMD:R_0805_2012Metric, F.Cu at (33.5, -12.6)
- added R21: R25, Resistor_SMD:R_0805_2012Metric, F.Cu at (56.5, 12.6)
- added R22: R25, Resistor_SMD:R_0805_2012Metric, F.Cu at (52.5, 12.6)
- added R23: R25, Resistor_SMD:R_0805_2012Metric, F.Cu at (15.5, 12.6)
- added R24: R25, Resistor_SMD:R_0805_2012Metric, F.Cu at (11.5, 12.6)
- added R47: R25, Resistor_SMD:R_0805_2012Metric, F.Cu at (11.5, -12.6)
- added R7: 330R, Resistor_SMD:R_0402_1005Metric, F.Cu at (24.1, 45.9)
- added R8: 330R, Resistor_SMD:R_0402_1005Metric, F.Cu at (34.2, 37.3)
- added REF**: PinSocket_1x40_P1.00mm_Vertical, Connector_PinSocket_1.00mm:PinSocket_1x40_P1.00mm_Vertical, F.Cu at (106.8, 16.9)
- added REF**: PinSocket_1x30_P1.27mm_Vertical, Connector_PinSocket_1.27mm:PinSocket_1x30_P1.27mm_Vertical, F.Cu at (100.9, 15.6)
- added REF**: MountingHole_3.2mm_M3, MountingHole:MountingHole_3.2mm_M3, F.Cu at (39.0, 10.0)
- added REF**: SolderJumper-3_P2.0mm_Open_TrianglePad1.0x1.5mm, Jumper:SolderJumper-3_P2.0mm_Open_TrianglePad1.0x1.5mm, F.Cu at (0.10, -1.93)
- added REF**: MountingHole_3.2mm_M3, MountingHole:MountingHole_3.2mm_M3, F.Cu at (82.0, 0.00)
- added REF**: MountingHole_3.2mm_M3, MountingHole:MountingHole_3.2mm_M3, F.Cu at (39.0, -10.0)
- C28, C29, C30, C69, C70, C71: footprint Capacitor_SMD:CP_Elec_8x6.7 -> Capacitor_SMD:CP_Elec_6.3x7.7
- J17, J18, J19, J20, J21, J22, J25, J26, P1, P2, P3, P4, P5, P6: moved to F.Cu
- moved J25 265.5 mm to (-4.33, -23.7), turned to 180 degrees
- moved J26 251.7 mm to (-18.2, 6.38)
- moved C19 246.7 mm to (14.5, -24.8)
- moved R97 246.7 mm to (13.0, -24.3)
- moved P1 233.0 mm to (10.0, -8.40)
- moved U5 231.3 mm to (13.5, -16.7)
- moved C49 231.2 mm to (17.1, -16.8)
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Routing:
- net +3V3: track 336.6 -> 128.8 mm, vias 8 -> 0
- net PC13: track 165.5 -> 28.4 mm, vias 8 -> 0
- net V_TMC: track 36.0 -> 149.3 mm, vias 65 -> 80
- net V_PWM_EB: track 99.5 -> 0.00 mm
- net PWM0_E3: track 89.1 -> 0.00 mm, vias 4 -> 0
- net GND_EB: track 77.3 -> 0.00 mm, vias 49 -> 0
- net 3V3_EB: track 75.7 -> 0.00 mm, vias 3 -> 0
- net ES4: track 64.7 -> 0.00 mm, vias 2 -> 0
- net V_SERVO: track 59.2 -> 0.00 mm, vias 6 -> 0
- net ES0: track 55.9 -> 0.00 mm, vias 4 -> 0
- net PWM1_E3: track 53.2 -> 0.00 mm, vias 3 -> 0
- net Net-(J2-Pad2): track 53.1 -> 0.00 mm, vias 2 -> 0
- net GND_EB_ADC: track 51.1 -> 0.00 mm, vias 1 -> 0
- net ES5: track 50.6 -> 0.00 mm, vias 2 -> 0
- net PA4: track 56.5 -> 6.64 mm, vias 2 -> 0
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- removed copper zone on F.Cu, net +3V3
- removed copper zone on In1.Cu, net GND
- removed copper zone on B.Cu, net GND_EB
- removed copper zone on F.Cu, net GND_EB
- removed copper zone on In1.Cu, net GND_EB
- removed copper zone on F.Cu, net GND_EB_ADC
- removed copper zone on F.Cu, net Net-(D4-Pad2)
- removed copper zone on F.Cu, net Net-(D5-Pad2)
- removed copper zone on F.Cu, net Net-(D6-Pad2)
- removed copper zone on F.Cu, net Net-(D9-Pad2)
- removed copper zone on F.Cu, net Net-(Q1-Pad1)
- removed copper zone on In2.Cu, net Net-(Q1-Pad1)
- removed copper zone on F.Cu, net Net-(Q2-Pad1)
- removed copper zone on In2.Cu, net Net-(Q2-Pad1)
- removed copper zone on F.Cu, net Net-(Q3-Pad1)
- removed copper zone on In2.Cu, net Net-(Q3-Pad1)
- removed copper zone on F.Cu, net Net-(Q4-Pad1)
- removed copper zone on In2.Cu, net Net-(Q4-Pad1)
- removed copper zone on F.Cu, net Net-(Q5-Pad1)
- removed copper zone on In2.Cu, net Net-(Q5-Pad1)
- removed copper zone on F.Cu, net PWM2_E3
- removed copper zone on In2.Cu, net PWM2_E3
- removed copper zone on F.Cu, net PWM3_E3
- removed copper zone on In2.Cu, net PWM3_E3
- removed copper zone on F.Cu, net V_PWM_EB
- removed copper zone on F.Cu, net V_SERVO
- removed copper zone on In2.Cu, net V_SERVO
- removed copper zone on In2.Cu, net V_TMC
Other:
- board size 213 x 95.1 mm -> 85.5 x 40 mm
- rule trace_min: 0.2 -> 0.15
- board text removed: "+"
- board text removed: "-"
- board text removed: "10A"
- board text removed: "15A"
- board text removed: "3V3"
- board text removed: "5A"
- board text removed: "<30V"
- board text removed: "ADC0"
- board text removed: "ADC1"
- board text removed: "E0"
- board text removed: "E1"
- board text removed: "E2"
- board text removed: "E3"
- board text removed: "E4"
- board text removed: "E5"
- board text removed: "GND"
- board text removed: "M0"
- board text removed: "M1"
- board text removed: "M2"
- board text removed: "M3"
- board text removed: "M4"
- board text removed: "M5"
- board text removed: "PA0"
- board text removed: "PA1"
- board text removed: "PA2"
- board text removed: "PA3"
- board text removed: "PA6"
- board text removed: "PA7"
- board text removed: "PB0"
- board text removed: "PB1"
- board text removed: "PB10"
- board text removed: "PB3"
- board text removed: "PB6"
- board text removed: "PB7"
- board text removed: "PWM0"
- board text removed: "PWM1"
- board text removed: "PWM2"
- board text removed: "PWM3"
- board text removed: "RX"
- board text removed: "S0"
- board text removed: "S1"
- board text removed: "SEN"
- board text removed: "SRC"
- board text removed: "TX"
- board text removed: "VCC"
- board text removed: "VSR"
- board text removed: "VST 5.5V-24V"
- board text removed: "s"
