File: MVSC2.kicad_pcb (KiCad board)
At the start: 4 copper layers, 85.5 x 40 mm, 206 parts, among them J1 USB_C-SIGNAL, J10 PWM3_OUT, J11 PWM_IN, J12 HSES, J16 ADC0, J17 ESTP0, J18 ESTP1, J19 ESTP2, J2 EXP0, J20 ESTP3, J21 ESTP4, J22 ESTP5, J23 POWER, J25 SERV0, J26 SERV1, J29 ADC1, J3 EXP1, J30 HSES, J31 HSES, J32 HSES, J4 EXPB, J5 HSES, J6 PWM0_OUT, J7 PWM1_OUT, J8 HSES, J9 PWM2_OUT, P1 STP0, P2 STP2, P3 STP4, P4 STP1, P5 STP3, P6 STP5, P9 UART, Q1 AO3400A, Q10 AO3400A, Q2 AO3400A, Q3 AO3400A, Q4 AO3400A, Q5 AO3400A, Q6 AO3400A, SW1 SKRKAEE020, SW2 SKRKAEE020, U1 XC6206P332MR, U10 TMC2208-LA-T, U11 TMC2208-LA-T, U12 TMC2208-LA-T, U13 CH912LSR, U14 CH912LSR, U2 CH912LSR, U3 STM32F411RET6, U4 CH912LSR, U5 TMC2208-LA-T, U6 TMC2208-LA-T, U7 TMC2208-LA-T, U8 CH912LSR, U9 CH912LSR, Y1 25MHZ 12pF, Y2 32.768KHz 12.5pF

Commit message: working layout - needs tripple checking
Parts:
- removed C120, C17, C2, C4: 100nF 16V, Capacitor_SMD:C_0402_1005Metric
- removed D1, D4, D5, D6, D9: B5819W, Diode_SMD:D_SOD-123
- removed J10: PWM3_OUT, Connector_JST:JST_PH_B2B-PH-K_1x02_P2.00mm_Vertical
- removed J11: PWM_IN, Connector_AMASS:AMASS_XT30U-M_1x02_P5.0mm_Vertical
- removed J12, J5, J8: HSES, Connector_PinHeader_1.00mm:PinHeader_1x03_P1.00mm_Vertical
- removed J25: SERV0, Connector_JST:JST_PH_B3B-PH-K_1x03_P2.00mm_Vertical
- removed J26: SERV1, Connector_JST:JST_PH_B3B-PH-K_1x03_P2.00mm_Vertical
- removed P9: UART, Connector_JST:JST_PH_B4B-PH-K_1x04_P2.00mm_Vertical
- removed R103, R104, R38, R41, R42, R43, R44: 330R, Resistor_SMD:R_0402_1005Metric
- removed the REF** at (106.8, 16.9)
- removed the REF** at (100.9, 15.6)
- removed the REF** at (0.10, -1.93)
- removed the REF** at (78.9, 74.4)
- removed the REF** at (178.0, 78.0)
- removed the REF** at (180.0, 78.0)
- removed TP1: SWD_DIO, TestPoint:TestPoint_THTPad_1.0x1.0mm_Drill0.5mm
- removed TP2: SWD_CLK, TestPoint:TestPoint_THTPad_1.0x1.0mm_Drill0.5mm
- removed TP3: SWD_GND, TestPoint:TestPoint_THTPad_1.0x1.0mm_Drill0.5mm
- removed U13, U14, U2: CH912LSR, Package_TO_SOT_SMD:SOT-23W
- added D13: Yellow, LED_SMD:LED_0603_1608Metric, F.Cu at (37.2, 16.6)
- added D7: Yellow, LED_SMD:LED_0603_1608Metric, F.Cu at (37.1, -14.9)
- added D8: Yellow, LED_SMD:LED_0603_1608Metric, F.Cu at (92.0, 15.5)
- added JP1: USB SRV SRC, Jumper:SolderJumper-2_P1.3mm_Open_TrianglePad1.0x1.5mm, F.Cu at (18.8, -1.52)
- added R25: 4.7k, Resistor_SMD:R_0402_1005Metric, F.Cu at (37.2, -17.1)
- added REF**: MountingHole_2.2mm_M2, MountingHole:MountingHole_2.2mm_M2, F.Cu at (100.0, 17.5)
- added REF**: MountingHole_2.2mm_M2, MountingHole:MountingHole_2.2mm_M2, F.Cu at (100.0, 3.63)
- added REF**: MountingHole_2.2mm_M2, MountingHole:MountingHole_2.2mm_M2, F.Cu at (100.0, -10.2)
- added REF**: MountingHole_3.2mm_M3, MountingHole:MountingHole_3.2mm_M3, F.Cu at (76.0, 10.0)
- added tooling: MountingHole_2.2mm_M2, MountingHole:MountingHole_2.2mm_M2, F.Cu at (10.3, 0.00)
- added tooling: MountingHole_2.2mm_M2, MountingHole:MountingHole_2.2mm_M2, F.Cu at (95.8, 19.0)
- added tooling: MountingHole_2.2mm_M2, MountingHole:MountingHole_2.2mm_M2, F.Cu at (95.8, -19.0)
- D3: value B5819W -> Yellow; footprint Diode_SMD:D_SOD-123 -> LED_SMD:LED_0603_1608Metric
- J16: value ADC0 -> ADC_HB
- J2: value EXP0 -> SWD; footprint Connector_PinHeader_2.00mm:PinHeader_1x08_P2.00mm_Vertical -> Connector_PinHeader_2.54mm:PinHeader_1x03_P2.54mm_Vertical
- J29: value ADC1 -> ADC_E
- J3: value EXP1 -> EXPP0; footprint Connector_PinHeader_2.00mm:PinHeader_1x08_P2.00mm_Vertical -> Connector_JST:JST_PH_B3B-PH-K_1x03_P2.00mm_Vertical
- J4: value EXPB -> EXPP1; footprint Connector_PinHeader_2.00mm:PinHeader_1x08_P2.00mm_Vertical -> Connector_JST:JST_PH_B6B-PH-K_1x06_P2.00mm_Vertical
- J6: value PWM0_OUT -> PWM_E
- J7: value PWM1_OUT -> PWM_HB
- J9: value PWM2_OUT -> PWM_FAN
- R12: value 330k -> 330R
- R29: value 5.1k -> 330R
- R37, R40, R7: value 330R -> 4.7k
- R8: value 330R -> 10k
- U3: value STM32F411RET6 -> STM32F411CEU6; footprint Package_QFP:LQFP-64_10x10mm_P0.5mm -> Package_DFN_QFN:QFN-48-1EP_7x7mm_P0.5mm_EP5.6x5.6mm
- moved R26 162.0 mm to (79.9, -17.7), turned to 180 degrees
- moved Q10 160.2 mm to (77.0, -16.5), turned to 270 degrees
- moved C26 149.0 mm to (82.0, -15.3), turned to 180 degrees
- moved R39 148.7 mm to (80.0, -15.3), turned to 180 degrees
- moved Q6 131.1 mm to (87.0, 3.50), turned to 270 degrees
- moved R12 130.6 mm to (87.1, 0.88), turned to 0 degrees
- moved R2 126.8 mm to (89.8, 0.88), turned to 0 degrees
- moved R11 126.1 mm to (92.4, 0.89), turned to 0 degrees
- moved Q4 125.9 mm to (92.0, -3.50), turned to 90 degrees
- moved Q3 120.8 mm to (92.0, 3.50), turned to 270 degrees
- moved R5 120.1 mm to (89.8, -0.91), turned to 180 degrees
- moved Q2 119.4 mm to (87.0, -16.5), turned to 270 degrees
- moved R9 116.2 mm to (87.1, -0.91), turned to 180 degrees
- moved Q1 115.7 mm to (87.0, -3.50), turned to 90 degrees
- moved R6 115.3 mm to (89.4, -17.2), turned to 90 degrees
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Connections:
- C25 pad 1: GND_EB_ADC -> GND
- C25 pad 2: ADC0 -> PA7
- C26 pad 1: GND_EB_ADC -> GND
- C26 pad 2: ADC1 -> PA3
- D2 pad 2: Net-(D2-Pad2) -> VBUS
- D3 pad 1: VBUS -> Net-(D3-Pad1)
- D3 pad 2: Net-(D3-Pad2) -> PA4
- J1 pad A4: Net-(D1-Pad2) -> VBUS
- J1 pad A9: Net-(D1-Pad2) -> VBUS
- J1 pad B4: Net-(D1-Pad2) -> VBUS
- J1 pad B9: Net-(D1-Pad2) -> VBUS
- J16 pad 1: GND_EB_ADC -> GND
- J16 pad 2: ADC0 -> PA7
- J17 pad 3: +3V3 -> V_EXP
- J18 pad 3: +3V3 -> V_EXP
- J19 pad 3: +3V3 -> V_EXP
- J2 pad 2: Net-(J2-Pad2) -> PA14
- J2 pad 3: Net-(J2-Pad3) -> PA13
- J20 pad 3: +3V3 -> V_EXP
- J21 pad 3: +3V3 -> V_EXP
- J22 pad 3: +3V3 -> V_EXP
- J23 pad 2: V_SERVO -> V_EXP
- J29 pad 1: GND_EB_ADC -> GND
- J29 pad 2: ADC1 -> PA3
- J3 pad 1: GND -> EXP0
- J3 pad 2: Net-(J3-Pad2) -> GND
- J3 pad 3: Net-(J3-Pad3) -> V_EXP
- J4 pad 1: GND_EB_ADC -> GND
- J4 pad 2: PWM3_E3 -> V_EXP
- J4 pad 3: PWM2_E3 -> EXP2
- J4 pad 4: ADC1 -> EXP4
- J4 pad 5: ADC0 -> EXP3
- J4 pad 6: PWM1_E3 -> EXP1
- J6 pad 1: Net-(D4-Pad2) -> GND1
- J6 pad 2: V_PWM_EB -> Net-(J6-Pad2)
- J7 pad 1: Net-(D5-Pad2) -> GND1
- J7 pad 2: V_PWM_EB -> Net-(J7-Pad2)
- J9 pad 1: Net-(D9-Pad2) -> GND1
- J9 pad 2: V_PWM_EB -> Net-(J9-Pad2)
- Q1 pad 2: GND_EB -> GND1
- Q1 pad 3: Net-(D4-Pad2) -> Net-(J6-Pad2)
- Q10 pad 1: PWM2_E3 -> EXP2
- Q10 pad 2: GND_EB -> GND1
- Q10 pad 3: Net-(D9-Pad2) -> Net-(J9-Pad2)
- Q2 pad 2: GND_EB -> GND1
- Q2 pad 3: Net-(D4-Pad2) -> Net-(J6-Pad2)
- Q3 pad 2: GND_EB -> GND1
- Q3 pad 3: Net-(D5-Pad2) -> Net-(J7-Pad2)
- Q4 pad 2: GND_EB -> GND1
- Q4 pad 3: Net-(D4-Pad2) -> Net-(J6-Pad2)
- Q5 pad 2: GND_EB -> GND1
- Q5 pad 3: Net-(D5-Pad2) -> Net-(J7-Pad2)
- Q6 pad 1: PWM3_E3 -> Net-(Q6-Pad1)
- Q6 pad 2: GND_EB -> GND1
- Q6 pad 3: Net-(D6-Pad2) -> Net-(J7-Pad2)
- R1 pad 1: PWM0_E3 -> PA4
- R1 pad 2: GND_EB -> GND1
- R10 pad 1: PWM1_E3 -> PA6
- R11 pad 1: PWM1_E3 -> PA6
- R12 pad 1: PWM3_E3 -> PA6
- R12 pad 2: GND_EB -> Net-(Q6-Pad1)
- R2 pad 1: PWM1_E3 -> PA6
- R2 pad 2: GND_EB -> GND1
- R26 pad 1: PWM2_E3 -> GND1
- R26 pad 2: GND_EB -> EXP2
- R29 pad 1: GND -> GND1
- R29 pad 2: Net-(D2-Pad1) -> GND
- R30 pad 2: Net-(D2-Pad2) -> PB2
- R31 pad 1: ADC0 -> PA7
- R31 pad 2: 3V3_EB -> +3V3
- R32 pad 1: PA6 -> PA3
- R32 pad 2: Net-(J3-Pad7) -> EXP0
- R33 pad 1: PA7 -> PA4
- R33 pad 2: Net-(J3-Pad6) -> EXP1
- R34 pad 1: PB0 -> PA5
- R34 pad 2: Net-(J3-Pad5) -> EXP2
- R35 pad 1: PB1 -> PA6
- R35 pad 2: Net-(J3-Pad4) -> EXP3
- R36 pad 1: PB10 -> PA7
- R36 pad 2: Net-(J3-Pad3) -> EXP4
- R37 pad 1: PB3 -> GND
- R37 pad 2: Net-(J3-Pad2) -> Net-(D3-Pad1)
- R39 pad 1: ADC1 -> PA3
- R39 pad 2: 3V3_EB -> +3V3
- R40 pad 1: PA2 -> GND
- R40 pad 2: Net-(J2-Pad5) -> Net-(D8-Pad1)
- R45 pad 1: PC13 -> PB1
- R5 pad 1: PWM0_E3 -> PA4
- R6 pad 1: PWM0_E3 -> PA4
- R7 pad 1: PA9 -> Net-(D2-Pad1)
- R7 pad 2: Net-(P9-Pad2) -> GND
- R8 pad 1: PA10 -> GND
- R9 pad 1: PWM0_E3 -> PA4
- U10 pad 19: PD2 -> PB3
- U10 pad 2: PC13 -> PB1
- U11 pad 14: PC9 -> PA8
- U11 pad 16: PC8 -> PB15
- U11 pad 19: PC7 -> PB14
- U11 pad 2: PC13 -> PB1
- U12 pad 14: PC4 -> PA2
- U12 pad 16: PC5 -> PA1
- U12 pad 19: PA4 -> PA0
- U12 pad 2: PC13 -> PB1
- U3 pad 10: PC2 -> PA0
- U3 pad 11: ES0 -> PA1
- U3 pad 12: GND -> PA2
- U3 pad 13: +3V3 -> PA3
- U3 pad 14: PA0 -> PA4
- U3 pad 15: PA1 -> PA5
- U3 pad 16: PA2 -> PA6
- U3 pad 17: PA3 -> PA7
- U3 pad 18: GND -> ES5
- U3 pad 19: +3V3 -> PB1
- U3 pad 20: PA4 -> PB2
- U3 pad 21: ES5 -> ES4
- U3 pad 22: PA6 -> Net-(C10-Pad1)
- U3 pad 23: PA7 -> GND
- U3 pad 24: PC4 -> +3V3
- U3 pad 25: PC5 -> PB12
- U3 pad 26: PB0 -> PB13
- U3 pad 27: PB1 -> PB14
- U3 pad 28: Net-(D2-Pad2) -> PB15
- U3 pad 29: PB10 -> PA8
- U3 pad 30: Net-(C10-Pad1) -> ES3
- U3 pad 31: GND -> ES2
- U3 pad 32: +3V3 -> USB_DN
- U3 pad 33: ES4 -> USB_DP
- U3 pad 34: PB13 -> PA13
- U3 pad 35: PB14 -> GND
- U3 pad 36: PB15 -> +3V3
- U3 pad 37: ES3 -> PA14
- U3 pad 38: PC7 -> PA15
- U3 pad 39: PC8 -> PB3
- U3 pad 40: PC9 -> PB4
- U3 pad 41: ES2 -> PB5
- U3 pad 42: PA9 -> ES1
- U3 pad 43: PA10 -> ES0
- U3 pad 44: USB_DN -> Net-(R17-Pad1)
- U3 pad 45: USB_DP -> PB8
- U3 pad 46: PA13 -> PB9
- U3 pad 49: PA14 -> GND
- U3 pad 8: PC0 -> GND
- U3 pad 9: PC1 -> +3V3
- U5 pad 14: PC0 -> PC13
- U5 pad 16: PC1 -> PB9
- U5 pad 19: PC2 -> PB8
- U5 pad 2: PC13 -> PB1
- U6 pad 14: PC11 -> PA15
- U6 pad 16: PC10 -> PA14
- U6 pad 19: PA15 -> PA13
- U6 pad 2: PC13 -> PB1
- U7 pad 14: PB15 -> PB12
- U7 pad 16: PB14 -> PB13
- U7 pad 19: PB13 -> PB2
- U7 pad 2: PC13 -> PB1
Routing:
- net +3V3: track 128.8 -> 432.0 mm, vias 0 -> 10
- net PB1: track 0.00 -> 180.7 mm, vias 0 -> 8
- net GND: track 255.1 -> 417.4 mm, vias 124 -> 121
- net PA4: track 6.64 -> 159.4 mm, vias 0 -> 3
- net EXP2: track 0.00 -> 146.1 mm, vias 0 -> 3
- net PA6: track 0.00 -> 109.8 mm, vias 0 -> 3
- net PA3: track 0.00 -> 101.6 mm, vias 0 -> 2
- net USB_DN: track 2.96 -> 80.3 mm, vias 0 -> 2
- net USB_DP: track 2.99 -> 76.9 mm, vias 0 -> 2
- net PA7: track 0.00 -> 66.1 mm, vias 0 -> 2
- net V_TMC: track 149.3 -> 194.0 mm, vias 80 -> 75
- net PB5: track 0.00 -> 44.0 mm, vias 0 -> 2
- net PC13: track 28.4 -> 71.7 mm
- net PA8: track 0.00 -> 40.7 mm
- net GND1: track 0.00 -> 37.1 mm, vias 0 -> 35
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- added copper zone on F.Cu, net +3V3
- added copper zone on In1.Cu, net GND
- added copper zone on B.Cu, net GND1
- added copper zone on F.Cu, net GND1
- added copper zone on In1.Cu, net GND1
- added copper zone on In2.Cu, net GND1
- added copper zone on F.Cu, net Net-(J6-Pad2)
- added copper zone on F.Cu, net Net-(J7-Pad2)
- added copper zone on F.Cu, net Net-(J9-Pad2)
- added copper zone on F.Cu, net V_EXP
- added copper zone on In1.Cu, net V_EXP
- added copper zone on In2.Cu, net V_TMC
Other:
- board size 85.5 x 40 mm -> 96 x 40 mm
- board text added: "-24V"
- board text added: "1"
- board text added: "ADC_E"
- board text added: "ADC_HB"
- board text added: "E0"
- board text added: "E1"
- board text added: "E2"
- board text added: "E3"
- board text added: "E4"
- board text added: "E5"
- board text added: "FAN"
- board text added: "GND"
- board text added: "IN"
- board text added: "IN -> PSU GND"
- board text added: "M0"
- board text added: "M1"
- board text added: "M2"
- board text added: "M3"
- board text added: "M4"
- board text added: "M5"
- board text added: "OUT"
- board text added: "OUT -> load GND (open drain)"
- board text added: "PWM_E"
- board text added: "PWM_HB"
- board text added: "SEN"
- board text added: "SWD"
- board text added: "VBUS"
- board text added: "VDD"
- board text added: "VEXP"
- board text added: "VEXP=5V"
- board text added: "VTMC"
- board text added: "VTMC=5.5V"
- board text added: "shorten leads; glue con.; solder top"

Commit message: fixed all drc errors and checked zones; still TODO: check everything
Routing:
- net V_TMC: track 194.0 -> 274.0 mm
- net GND: track 417.4 -> 487.6 mm, vias 121 -> 120
- net V_EXP: track 29.8 -> 41.8 mm
- net +3V3: track 432.0 -> 426.7 mm

Commit message: working version with mosfets
Parts:
- added G***: LOGO, MVSC2:logo, F.Cu at (35.5, 3.75)
- moved e 1.00 mm to (95.8, -18.0)
- moved tooling 1.00 mm to (95.8, 18.0)
- renumbered tooling to e
Routing:
- net V_EXP: track 41.8 -> 67.6 mm
- net GND: track 487.6 -> 488.5 mm
Other:
- board text added: "MVSC2"
- board text added: "VEXP: 5V"
- board text added: "VTMC: 5.5V"
- board text added: "v0"
- board text removed: "VEXP=5V"
- board text removed: "VTMC=5.5V"
