File: MVSC2.kicad_pcb (KiCad board)
At the start: 4 copper layers, 96 x 40 mm, 183 parts, among them J1 USB_C-SIGNAL, J16 ADC_HB, J17 ESTP0, J18 ESTP1, J19 ESTP2, J2 SWD, J20 ESTP3, J21 ESTP4, J22 ESTP5, J23 POWER, J29 ADC_E, J3 EXPP0, J30 HSES, J31 HSES, J32 HSES, J4 EXPP1, J6 PWM_E, J7 PWM_HB, J9 PWM_FAN, P1 STP0, P2 STP2, P3 STP4, P4 STP1, P5 STP3, P6 STP5, Q1 AO3400A, Q10 AO3400A, Q2 AO3400A, Q3 AO3400A, Q4 AO3400A, Q5 AO3400A, Q6 AO3400A, SW1 SKRKAEE020, SW2 SKRKAEE020, U1 XC6206P332MR, U10 TMC2208-LA-T, U11 TMC2208-LA-T, U12 TMC2208-LA-T, U3 STM32F411CEU6, U4 CH912LSR, U5 TMC2208-LA-T, U6 TMC2208-LA-T, U7 TMC2208-LA-T, U8 CH912LSR, U9 CH912LSR, Y1 25MHZ 12pF, Y2 32.768KHz 12.5pF

Commit message: final, ordered
Parts:
- removed C25, C26: 4.7uF 10V, Capacitor_SMD:C_0402_1005Metric
- removed D3, D8: Yellow, LED_SMD:LED_0603_1608Metric
- removed J16: ADC_HB, Connector_JST:JST_PH_B2B-PH-K_1x02_P2.00mm_Vertical
- removed J29: ADC_E, Connector_JST:JST_PH_B2B-PH-K_1x02_P2.00mm_Vertical
- removed J6: PWM_E, Connector_AMASS:AMASS_XT30U-F_1x02_P5.0mm_Vertical
- removed J7: PWM_HB, Connector_AMASS:AMASS_XT30U-F_1x02_P5.0mm_Vertical
- removed J9: PWM_FAN, Connector_JST:JST_PH_B2B-PH-K_1x02_P2.00mm_Vertical
- removed Q1, Q10, Q2, Q3, Q4, Q5, Q6: AO3400A, Package_TO_SOT_SMD:SOT-23W
- removed R1, R2, R26: 330k, Resistor_SMD:R_0402_1005Metric
- removed R10, R11, R12, R29, R5, R6, R9: 330R, Resistor_SMD:R_0402_1005Metric
- removed R31, R37, R39, R40: 4.7k, Resistor_SMD:R_0402_1005Metric
- removed the REF** at (76.0, 10.0)
- removed the REF** at (71.0, -10.0)
- moved G*** 36.7 mm to (69.8, -9.13), turned to 90 degrees
- moved C27 23.0 mm to (79.2, -15.5)
- moved C52 23.0 mm to (79.2, 12.2)
- moved C68 23.0 mm to (79.2, -1.67)
- moved D10 23.0 mm to (74.4, -14.7)
- moved D11 23.0 mm to (74.4, 12.9)
- moved D12 23.0 mm to (74.4, -0.91)
- moved J30 23.0 mm to (75.0, -18.0)
- moved J31 23.0 mm to (75.0, 9.66)
- moved J32 23.0 mm to (75.0, -4.17)
- moved REF** 23.0 mm to (77.0, 17.5)
- moved REF** 23.0 mm to (77.0, 3.63)
- moved REF** 23.0 mm to (77.0, -10.2)
- moved U4 23.0 mm to (77.0, -14.6)
- moved U8 23.0 mm to (77.0, 13.1)
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Connections:
- net EXP0 renamed Net-(J3-Pad1)
- net EXP1 renamed Net-(J4-Pad6)
- net EXP2 renamed Net-(J4-Pad3)
- net EXP3 renamed Net-(J4-Pad5)
- net EXP4 renamed Net-(J4-Pad4)
Routing:
- net Net-(J4-Pad3): track 146.1 -> 48.5 mm, vias 3 -> 2
- net PA4: track 159.4 -> 63.7 mm, vias 3 -> 2
- net +3V3: track 426.7 -> 343.0 mm, vias 10 -> 8
- net PA6: track 109.8 -> 28.3 mm, vias 3 -> 2
- net GND: track 488.5 -> 411.9 mm, vias 120 -> 118
- net GND1: track 37.1 -> 0.00 mm, vias 35 -> 0
- net PA3: track 101.6 -> 65.4 mm
- net PA7: track 66.1 -> 41.2 mm
- net Net-(J6-Pad2): track 20.7 -> 0.00 mm
- net Net-(J7-Pad2): track 20.4 -> 0.00 mm
- net Net-(J9-Pad2): track 7.79 -> 0.00 mm
- net Net-(Q4-Pad1): track 2.70 -> 0.00 mm
- net Net-(Q1-Pad1): track 1.81 -> 0.00 mm
- net Net-(D8-Pad1): track 1.77 -> 0.00 mm
- net Net-(D3-Pad1): track 1.69 -> 0.00 mm
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- removed copper zone on B.Cu, net GND1
- removed copper zone on F.Cu, net GND1
- removed copper zone on In1.Cu, net GND1
- removed copper zone on In2.Cu, net GND1
- removed copper zone on F.Cu, net Net-(J6-Pad2)
- removed copper zone on F.Cu, net Net-(J7-Pad2)
- removed copper zone on F.Cu, net Net-(J9-Pad2)
Other:
- board size 96 x 40 mm -> 73 x 40 mm
- board text added: "VCC"
- board text removed: "ADC_E"
- board text removed: "ADC_HB"
- board text removed: "FAN"
- board text removed: "IN"
- board text removed: "IN -> PSU GND"
- board text removed: "OUT"
- board text removed: "OUT -> load GND (open drain)"
- board text removed: "PWM_E"
- board text removed: "PWM_HB"
- board text removed: "VDD"
