File: MVSC2.sch (KiCad schematic (older format))
At the start: 308 parts, among them J1 USB_C-SIGNAL, J10 PWM3_OUT, J11 PWM_IN, J12 EXP-1, J13 Exp2-smd, J14 EXP-3, J15 EXP-2, J16 ADC0, J17 ESTP0, J18 ESTP1, J19 ESTP2, J2 SERV2, J20 ESTP3, J21 ESTP4, J22 ESTP5, J23 POWER, J24 CaEx2, J25 SERV0, J26 SERV1, J27 CaEx2, J28 CaEx3, J29 ADC1, J3 EXP0, J30 HSES, J31 HSES, J32 HSES, J33 CaEx3, J34 SERV3, J35 SERV4, J36 SERV5, J37 EXP-SERVO, J38 I2C, J39 UART_pin, J4 EXP1, J40 UART, J41 I2C_pin, J42 I2C, J5 UART, J6 PWM0_OUT, J7 PWM1_OUT, J8 Exp1-pin, J9 PWM2_OUT, P1 STP0, P2 STP2, P3 STP4, P4 STP1, P5 STP3, P6 STP5, P7 CaEx4, P8 CaEx4, Q1 AO3400A, Q10 AO3400A, Q2 AO3400A, Q3 AO3400A, Q4 AO3400A, Q5 AO3400A, Q6 AO3400A, SW1 SKRKAEE020, SW2 SKRKAEE020, U1 XC6206P332MR, U10 TMC2208-LA-T, U11 TMC2208-LA-T, U12 TMC2208-LA-T, U3 STM32F411RCT6, U4 CH912LSR, U5 TMC2208-LA-T, U6 TMC2208-LA-T, U7 TMC2208-LA-T, U8 CH912LSR, U9 CH912LSR, Y1 25MHZ 12pF, Y2 32.768KHz 12.5pF

Commit message: working
Parts:
- removed C120, C121, C2, C4: 4.7uF 10V, Capacitor_SMD:C_0402_1005Metric, symbol Device:C
- removed J12: EXP-1, Connector_FFC-FPC:Hirose_FH12-20S-0.5SH_1x20-1MP_P0.50mm_Horizontal, symbol Connector_Generic:Conn_01x20
- removed J13: Exp2-smd, Connector_PinHeader_2.00mm:PinHeader_1x11_P2.00mm_Horizontal, symbol Connector_Generic:Conn_01x11
- removed J14: EXP-3, Connector_FFC-FPC:Hirose_FH12-20S-0.5SH_1x20-1MP_P0.50mm_Horizontal, symbol Connector_Generic:Conn_01x20
- removed J15: EXP-2, Connector_FFC-FPC:Hirose_FH12-20S-0.5SH_1x20-1MP_P0.50mm_Horizontal, symbol Connector_Generic:Conn_01x20
- removed J2: SERV2, Connector_JST:JST_PH_B3B-PH-K_1x03_P2.00mm_Vertical, symbol Connector_Generic:Conn_01x03
- removed J24, J27: CaEx2, Connector_JST:JST_PH_B2B-PH-K_1x02_P2.00mm_Vertical, symbol Connector_Generic:Conn_01x02
- removed J28, J33: CaEx3, Connector_JST:JST_PH_B3B-PH-K_1x03_P2.00mm_Vertical, symbol Connector_Generic:Conn_01x03
- removed J3: EXP0, Connector_FFC-FPC:Hirose_FH12-20S-0.5SH_1x20-1MP_P0.50mm_Horizontal, symbol Connector_Generic:Conn_01x20
- removed J34: SERV3, Connector_JST:JST_PH_B3B-PH-K_1x03_P2.00mm_Vertical, symbol Connector_Generic:Conn_01x03
- removed J35: SERV4, Connector_JST:JST_PH_B3B-PH-K_1x03_P2.00mm_Vertical, symbol Connector_Generic:Conn_01x03
- removed J36: SERV5, Connector_JST:JST_PH_B3B-PH-K_1x03_P2.00mm_Vertical, symbol Connector_Generic:Conn_01x03
- removed J37: EXP-SERVO, Connector_FFC-FPC:Hirose_FH12-20S-0.5SH_1x20-1MP_P0.50mm_Horizontal, symbol Connector_Generic:Conn_01x20
- removed J38, J42: I2C, Connector_FFC-FPC:Hirose_FH12-6S-0.5SH_1x06-1MP_P0.50mm_Horizontal, symbol Connector_Generic:Conn_01x06
- removed J39: UART_pin, Connector_PinHeader_2.54mm:PinHeader_1x04_P2.54mm_Vertical, symbol Connector_Generic:Conn_01x04
- removed J4: EXP1, Connector_FFC-FPC:Hirose_FH12-20S-0.5SH_1x20-1MP_P0.50mm_Horizontal, symbol Connector_Generic:Conn_01x20
- removed J40, J5: UART, Connector_FFC-FPC:Hirose_FH12-6S-0.5SH_1x06-1MP_P0.50mm_Horizontal, symbol Connector_Generic:Conn_01x06
- removed J41: I2C_pin, Connector_PinHeader_2.54mm:PinHeader_1x04_P2.54mm_Vertical, symbol Connector_Generic:Conn_01x04
- removed J8: Exp1-pin, Connector_PinHeader_2.54mm:PinHeader_1x11_P2.54mm_Vertical, symbol Connector_Generic:Conn_01x11
- removed JP1, JP2, JP3, JP4, JP5, JP6, JP7, JP8: SJ_O, Jumper:SolderJumper-2_P1.3mm_Open_RoundedPad1.0x1.5mm, symbol Jumper:SolderJumper_2_Open
- removed P7, P8: CaEx4, Connector_JST:JST_PH_B4B-PH-K_1x04_P2.00mm_Vertical, symbol Connector_Generic:Conn_01x04
- removed R13, R14, R15, R16: 4.7k, Resistor_SMD:R_0402_1005Metric, symbol Device:R
- added J2: EXP0, Connector_PinHeader_2.00mm:PinHeader_1x08_P2.00mm_Vertical, symbol Connector_Generic:Conn_01x08
- added J3: EXP1, Connector_PinHeader_2.00mm:PinHeader_1x08_P2.00mm_Vertical, symbol Connector_Generic:Conn_01x08
- added J4: EXPB, Connector_PinHeader_2.00mm:PinHeader_1x08_P2.00mm_Vertical, symbol Connector_Generic:Conn_01x08
- added P9: UART, Connector_JST:JST_PH_B4B-PH-K_1x04_P2.00mm_Vertical, symbol Connector_Generic:Conn_01x04
- C1, C12, C3: LCSC (none) -> C52923
- C10, C11, C25, C26, C53, C54, C55, C93, C94, C95: LCSC (none) -> C23733
- C100, C101, C102, C103, C104, C105, C106, C107, C19, C20, C21, C22, C23, C24, C56, C57, C58, C59, C60, C61, C62, C63, C64, C65, C66, C67, C96, C97, C98, C99: LCSC (none) -> C1537
- C108, C109, C110, C111, C112, C113, C114, C115, C116, C117, C118, C119, C43, C44, C45, C46, C47, C48, C84, C85, C86, C87, C88, C89: LCSC (none) -> C1585
- C13, C14, C15, C16, C17, C18, C27, C31, C32, C33, C34, C35, C36, C37, C38, C39, C40, C41, C42, C52, C68, C72, C73, C74, C75, C76, C77, C78, C79, C80, C81, C82, C83, C9: LCSC (none) -> C1525
- C28, C29, C30, C69, C70, C71: LCSC (none) -> C250061
- C49, C50, C51, C90, C91, C92: LCSC (none) -> C1532
- C5, C6, C7, C8: LCSC (none) -> C1548
- D1, D3, D4, D5, D6, D9: LCSC (none) -> C8598
- D10, D11, D12, D2: LCSC (none) -> C72041
- Q1, Q10, Q2, Q3, Q4, Q5, Q6: LCSC (none) -> C20917
- R1, R12, R2, R26: LCSC (none) -> C25778
- R10, R100, R101, R102, R103, R104, R11, R32, R33, R34, R35, R36, R37, R38, R40, R41, R42, R43, R44, R5, R6, R7, R8, R9, R97, R98, R99: LCSC (none) -> C25104
- R17, R30: LCSC (none) -> C25779
- R29, R3, R4, R46, R71, R72: LCSC (none) -> C25905
- R31, R39: LCSC (none) -> C25900
- R45: LCSC (none) -> C25744
- R47, R48, R49, R50, R51, R52, R53, R54, R55, R56, R57, R58, R59, R60, R61, R62, R63, R64, R65, R66, R67, R68, R69, R70, R73, R74, R75, R76, R77, R78, R79, R80, R81, R82, R83, R84, R85, R86, R87, R88, R89, R90, R91, R92, R93, R94, R95, R96: LCSC (none) -> C25086
- SW1, SW2: LCSC (none) -> C115357
- U1: LCSC (none) -> C5446
- U10, U11, U12, U5, U6, U7: LCSC (none) -> C115944
- U3: value STM32F411RCT6 -> STM32F411RET6; LCSC (none) -> C94355
- U4, U8, U9: LCSC (none) -> C455294
- Y1: LCSC (none) -> C9006
- Y2: LCSC (none) -> C32346
Connections:
- net +3V3: now also J2.8 (Pin_8)
- net ADC0: now also J4.5 (Pin_5)
- net ADC1: now also J4.4 (Pin_4)
- net GND: now also J2.1 (Pin_1), J3.1 (Pin_1), P9.1 (Pin_1)
- net PWM0_E3: now also J4.7 (Pin_7)
- net PWM1_E3: now also J4.6 (Pin_6)
- net PWM2_E3: now also J4.3 (Pin_3)
- net PWM3_E3: now also J4.2 (Pin_2)
- net V_SERVO: now also J3.8 (Pin_8)
- net at D3.2 (A): now also P9.4 (Pin_4)
- net at R7.2: now also P9.2 (Pin_2)
- net at R8.2: now also P9.3 (Pin_3)
- net at R34.2: now also J3.5 (Pin_5)
- net at R35.2: now also J3.4 (Pin_4)
- net at R36.2: now also J3.3 (Pin_3)
- net at R37.2: now also J3.2 (Pin_2)
- net at R32.2: now also J3.7 (Pin_7)
- net at R33.2: now also J3.6 (Pin_6)
- net at R40.2: now also J2.5 (Pin_5)
- net at R41.2: now also J2.4 (Pin_4)
- net at R43.2: now also J2.3 (Pin_3)
- net at R44.2: now also J2.2 (Pin_2)
- net at R42.2: now also J2.6 (Pin_6)
- net at R38.2: now also J2.7 (Pin_7)
- net 3v3_E3 renamed 3V3_EB
- net 3V3_EB: now also J4.8 (Pin_8)
- net ADCGND_E3 renamed GND_EB_ADC
- net GND_EB_ADC: now also J4.1 (Pin_1)
- net GND_E3 renamed GND_EB
- net V_PWM_E3 renamed V_PWM_EB
- no-connect marks 64 -> 58
Other:
- note added: "0402WGF3303TCE\n0402"
- note added: "EXPANSION BOARD"
- note added: "separate gnd\nto prevent\nground loops"
- note removed: "CABLE EXTENSIONS"
- note removed: "EXPANSION BOARD 0"
- note removed: "EXPANSION BOARD 1"
- note removed: "EXPANSION BOARD 2"
- note removed: "EXPANSION BOARD 3"
- note removed: "I2C_SCL, PWM"
- note removed: "I2C_SDA, PWM"
- note removed: "Optional for ADC"
- note removed: "To prevent\nground loops"
- note removed: "Use any\ndirection cable"
- note removed: "Use reversed\ndirection cable"
- note removed: "With ribbon 0.5mm\ntotal max exp servo\ncurrent is 3A per\ncon."
- moved on the sheet: C25, C26, C27, C52, C68, D10, D11, D12, D3, D4, D5, D6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

Commit message: working
Parts:
- added C120, C2, C4: 100nF 16V, Capacitor_SMD:C_0402_1005Metric, symbol Device:C
- added J12, J5, J8: HSES, Connector_PinHeader_1.00mm:PinHeader_1x03_P1.00mm_Vertical, symbol Connector_Generic:Conn_01x03
- added U13, U14, U2: CH912LSR, Package_TO_SOT_SMD:SOT-23W, symbol Sensor_Magnetic:A1301KLHLT-T
Connections:
- new net: J12.1 (Pin_1), U14.2 (VOUT)
- new net: C120.2, J12.2 (Pin_2), U14.3 (GND)
- new net: C120.1, J12.3 (Pin_3), U14.1 (VCC)
- new net: J8.1 (Pin_1), U13.2 (VOUT)
- new net: C4.2, J8.2 (Pin_2), U13.3 (GND)
- new net: C4.1, J8.3 (Pin_3), U13.1 (VCC)
- new net: J5.1 (Pin_1), U2.2 (VOUT)
- new net: C2.2, J5.2 (Pin_2), U2.3 (GND)
- new net: C2.1, J5.3 (Pin_3), U2.1 (VCC)

Commit message: partial
Parts:
- removed C100, C101, C102, C103, C104, C105, C106, C107, C56, C57, C58, C59, C60, C61, C62, C63, C64, C65, C66, C67, C96, C97, C98, C99: 470pF 50V, Capacitor_SMD:C_0402_1005Metric, symbol Device:C
- removed C109, C110, C111, C115, C116, C117, C43, C44, C45, C84, C85, C86: 33nF 50V, Capacitor_SMD:C_0402_1005Metric, symbol Device:C
- removed C31, C33, C35, C37, C38, C39, C72, C74, C76, C78, C79, C80: 100nF 16V, Capacitor_SMD:C_0402_1005Metric, symbol Device:C
- removed R48, R49, R50, R51, R52, R53, R54, R55, R56, R57, R58, R59, R60, R61, R62, R63, R64, R65, R66, R67, R68, R69, R70, R73, R74, R75, R76, R77, R78, R79, R80, R81, R82, R83, R84, R85, R86, R87, R88, R89, R90, R91, R92, R93, R94, R95, R96: 1R, Resistor_SMD:R_0402_1005Metric, symbol Device:R
- added R13, R14, R15, R16, R18, R19, R20, R21, R22, R23, R24: R25, Resistor_SMD:R_0805_2012Metric, symbol Device:R
- C108, C112, C113, C114, C118, C119, C46, C47, C48, C87, C88, C89: value 33nF 50V -> 100nF 50V; footprint Capacitor_SMD:C_0402_1005Metric -> Capacitor_SMD:C_0603_1608Metric; LCSC C1585 -> C14663
- C28, C29, C30, C69, C70, C71: footprint Capacitor_SMD:CP_Elec_8x6.7 -> Capacitor_SMD:CP_Elec_6.3x7.7; LCSC C250061 -> C250084
- R47: value 1R -> R25; footprint Resistor_SMD:R_0402_1005Metric -> Resistor_SMD:R_0805_2012Metric; LCSC C25086 -> C46216
Connections:
- net GND: now also R13.1, R14.1, R15.1, R16.1, R18.1, R19.1, R20.1, R21.1, R22.1, R23.1, R24.1
- net at U10.23 (BRA): now also R19.2
- net at U10.27 (BRB): now also R20.2
- net at U11.23 (BRA): now also R21.2
- net at U11.27 (BRB): now also R22.2
- net at U12.23 (BRA): now also R23.2
- net at U12.27 (BRB): now also R24.2
- net at U5.27 (BRB): now also R13.2
- net at U6.23 (BRA): now also R14.2
- net at U6.27 (BRB): now also R15.2
- net at U7.23 (BRA): now also R16.2
- net at U7.27 (BRB): now also R18.2
Other:
- note added: "0805W8F250LT5F\n0805\n0.125W"
- note added: "CC0603KRX7R9BB104\n0603"
- note added: "Extended parts:\nSTM32F411RCT6\nTMC2208-LA-T\n1206W4F250LT5E\nOVZ101M1ETR-0608\nSKRKAEE020\nCH912LSR"
- note added: "OVZ101M1ETR-0608\nSMD-ECAP-6.3x7.7\nLOW ESR"
- note added: "RSense=0.25"
- note removed: "(I use 2x 33n instead of 1x 100n\nbecause jlcpcb and basic parts:\ntheir 100n 50V basic is 0603, not\n0402... which I want for layout\ndesign)"
- note removed: "0402B471K500NT\n0402"
- note removed: "0402F333M500NT\n0402"
- note removed: "0402WGF100KTCE\n0402\n0.0625W"
- note removed: "Extended parts:\nSTM32F411RCT6\nTMC2208-LA-T\nOVK101M1ETR-0807\nSKRKAEE020\nCH912LSR"
- note removed: "For RSENSE I want 0R25,\nbut on jlcpcb thats extended,\nits cheaper to put 4x R1 in\nparallel..."
- note removed: "OVK101M1ETR-0807\nSMD-ECAP-8.3x6.7\nLOW ESR"
- note removed: "RSense=0.25\n0.25W"
- moved on the sheet: R47

Commit message: working layout - needs tripple checking
Parts:
- removed C120, C17, C2, C4: 100nF 16V, Capacitor_SMD:C_0402_1005Metric, symbol Device:C
- removed D1, D3, D4, D5, D6, D9: B5819W, Diode_SMD:D_SOD-123, symbol Device:D_Schottky
- removed J10: PWM3_OUT, Connector_JST:JST_PH_B2B-PH-K_1x02_P2.00mm_Vertical, symbol Connector_Generic:Conn_01x02
- removed J11: PWM_IN, Connector_AMASS:AMASS_XT30U-M_1x02_P5.0mm_Vertical, symbol Connector_Generic:Conn_01x02
- removed J12, J5, J8: HSES, Connector_PinHeader_1.00mm:PinHeader_1x03_P1.00mm_Vertical, symbol Connector_Generic:Conn_01x03
- removed J2: EXP0, Connector_PinHeader_2.00mm:PinHeader_1x08_P2.00mm_Vertical, symbol Connector_Generic:Conn_01x08
- removed J25: SERV0, Connector_JST:JST_PH_B3B-PH-K_1x03_P2.00mm_Vertical, symbol Connector_Generic:Conn_01x03
- removed J26: SERV1, Connector_JST:JST_PH_B3B-PH-K_1x03_P2.00mm_Vertical, symbol Connector_Generic:Conn_01x03
- removed J3: EXP1, Connector_PinHeader_2.00mm:PinHeader_1x08_P2.00mm_Vertical, symbol Connector_Generic:Conn_01x08
- removed J4: EXPB, Connector_PinHeader_2.00mm:PinHeader_1x08_P2.00mm_Vertical, symbol Connector_Generic:Conn_01x08
- removed P9: UART, Connector_JST:JST_PH_B4B-PH-K_1x04_P2.00mm_Vertical, symbol Connector_Generic:Conn_01x04
- removed R103, R104, R38, R41, R42, R43, R44: 330R, Resistor_SMD:R_0402_1005Metric, symbol Device:R
- removed TP1: SWD_DIO, TestPoint:TestPoint_THTPad_1.0x1.0mm_Drill0.5mm, symbol Connector:TestPoint
- removed TP2: SWD_CLK, TestPoint:TestPoint_THTPad_1.0x1.0mm_Drill0.5mm, symbol Connector:TestPoint
- removed TP3: SWD_GND, TestPoint:TestPoint_THTPad_1.0x1.0mm_Drill0.5mm, symbol Connector:TestPoint
- removed U13, U14, U2: CH912LSR, Package_TO_SOT_SMD:SOT-23W, symbol Sensor_Magnetic:A1301KLHLT-T
- removed U3: STM32F411RET6, Package_QFP:LQFP-64_10x10mm_P0.5mm, symbol MCU_ST_STM32F4:STM32F411RCTx
- added D13, D3, D7, D8: Yellow, LED_SMD:LED_0603_1608Metric, symbol Device:LED
- added J2: SWD, Connector_PinHeader_2.54mm:PinHeader_1x03_P2.54mm_Vertical, symbol Connector_Generic:Conn_01x03
- added J3: EXPP0, Connector_JST:JST_PH_B3B-PH-K_1x03_P2.00mm_Vertical, symbol Connector_Generic:Conn_01x03
- added J4: EXPP1, Connector_JST:JST_PH_B6B-PH-K_1x06_P2.00mm_Vertical, symbol Connector_Generic:Conn_01x06
- added JP1: USB SRV SRC, Jumper:SolderJumper-2_P1.3mm_Open_TrianglePad1.0x1.5mm, symbol Jumper:SolderJumper_2_Open
- added R25: 4.7k, Resistor_SMD:R_0402_1005Metric, symbol Device:R
- added U3: STM32F411CEU6, Package_DFN_QFN:QFN-48-1EP_7x7mm_P0.5mm_EP5.6x5.6mm, symbol MCU_ST_STM32F4:STM32F411CEUx
- J16: value ADC0 -> ADC_HB
- J17, J18, J19, J20, J21, J22: Field5 SEN -> SIG
- J29: value ADC1 -> ADC_E
- J6: value PWM0_OUT -> PWM_E; Field4 + -> OUT; Field5 - -> IN
- J7: value PWM1_OUT -> PWM_HB; Field4 + -> OUT; Field5 - -> IN
- J9: value PWM2_OUT -> PWM_FAN; Field4 + -> OUT; Field5 - -> IN
- R12: value 330k -> 330R; LCSC C25778 -> C25104
- R29: value 5.1k -> 330R; LCSC C25905 -> C25104
- R37, R40, R7: value 330R -> 4.7k; LCSC C25104 -> C25900
- R8: value 330R -> 10k; LCSC C25104 -> C25744
Connections:
- net 3V3_EB is gone; now on net +3V3: R31.2, R39.2
- net ADC0 is gone; now on net PA7: C25.2, J16.2 (Pin_2), R31.1
- net ADC1 is gone; now on net PA3: C26.2, J29.2 (Pin_2), R39.1
- net GND_EB_ADC is gone; now on net GND: C25.1, C26.1, J16.1 (Pin_1), J29.1 (Pin_1)
- net PA10 is gone; now on net GND: R8.1
- net PA9 is gone; now on an unnamed net: R7.1
- net PB10 is gone; now on net PA7: R36.1
- net PC0 is gone; now on net PC13: U5.14 (PDN_UART)
- net PC1 is gone; now on net PB9: U5.16 (STEP)
- net PC10 is gone; now on net PA14: U6.16 (STEP)
- net PC11 is gone; now on net PA15: U6.14 (PDN_UART)
- net PC2 is gone; now on net PB8: U5.19 (DIR)
- net PC4 is gone; now on net PA2: U12.14 (PDN_UART)
- net PC5 is gone; now on net PA1: U12.16 (STEP)
- net PC7 is gone; now on net PB14: U11.19 (DIR)
- net PC8 is gone; now on net PB15: U11.16 (STEP)
- net PD2 is gone; now on net PB3: U10.19 (DIR)
- net PWM0_E3 is gone; now on net PA4: R1.1, R5.1, R6.1, R9.1
- net PWM1_E3 is gone; now on net PA6: R10.1, R11.1, R2.1
- net +3V3: now also U3.1 (VBAT), U3.24 (VDD), U3.36 (VDD), U3.48 (VDD), U3.9 (VDDA); no longer J17.3 (Pin_3), J18.3 (Pin_3), J19.3 (Pin_3), J20.3 (Pin_3), J21.3 (Pin_3), J22.3 (Pin_3)
- net ES0: now also U3.43 (PB7)
- net ES1: now also U3.42 (PB6)
- net ES2: now also U3.31 (PA10)
- net ES3: now also U3.30 (PA9)
- net ES4: now also U3.21 (PB10)
- net ES5: now also U3.18 (PB0)
- net GND: now also R29.2, R37.1, R40.1, R7.2, J2.1 (Pin_1), J3.2 (Pin_2), J4.1 (Pin_1), R25.2, U3.23 (VSS), U3.35 (VSS), U3.47 (VSS), U3.49 (VSS), U3.8 (VSSA); no longer R29.1
- net PA0: now also U12.19 (DIR), U3.10 (PA0)
- net PA1: now also U3.11 (PA1)
- net PA13: now also U6.19 (DIR), J2.3 (Pin_3), U3.34 (PA13)
- net PA14: now also J2.2 (Pin_2), U3.37 (PA14)
- net PA15: now also U3.38 (PA15); no longer U6.19 (DIR)
- net PA2: now also U3.12 (PA2); no longer R40.1
- net PA3: now also R32.1, U3.13 (PA3)
- net PA4: now also R33.1, D3.2 (A), U3.14 (PA4); no longer U12.19 (DIR)
- net PA6: now also R12.1, R35.1, D8.2 (A), U3.16 (PA6); no longer R32.1
- net PA7: now also U3.17 (PA7); no longer R33.1
- net PB1: now also R45.1, U10.2 (ENN), U11.2 (ENN), U12.2 (ENN), U5.2 (ENN), U6.2 (ENN), U7.2 (ENN), U3.19 (PB1); no longer R35.1
- net PB13: now also U7.16 (STEP), U3.26 (PB13); no longer U7.19 (DIR)
- net PB14: now also U3.27 (PB14); no longer U7.16 (STEP)
- net PB15: now also U3.28 (PB15); no longer U7.14 (PDN_UART)
- net PB3: now also U3.39 (PB3); no longer R37.1
- net PB4: now also U3.40 (PB4)
- net PB5: now also U3.41 (PB5)
- net PB8: now also U3.45 (PB8)
- net PB9: now also U3.46 (PB9)
- net PC13: now also U3.2 (PC13); no longer R45.1, U10.2 (ENN), U11.2 (ENN), U12.2 (ENN), U5.2 (ENN), U6.2 (ENN), U7.2 (ENN)
- net USB_DN: now also U3.32 (PA11)
- net USB_DP: now also U3.33 (PA12)
- net VBUS: now also D2.2 (A), J1.A4 (VBUS), J1.A9 (VBUS), J1.B4 (VBUS), J1.B9 (VBUS), JP1.1 (A)
- net V_TMC: now also D13.2 (A)
- net PB2: now reaches R30.2
- net PB2: now also U7.19 (DIR), U3.20 (PB2); no longer D2.2 (A)
- net at C7.2, Y2.2: now also U3.3 (PC14)
- net at C10.1: now also U3.22 (VCAP1)
- net at C8.2, Y2.1: now also U3.4 (PC15)
- net at C5.2, Y1.1: now also U3.5 (PH0)
- net at C6.2, Y1.3: now also U3.6 (PH1)
- net at R17.1, SW2.2: now also U3.44 (BOOT0)
- net at C9.1, SW1.2: now also U3.7 (NRST)
- net at R37.2: now also D3.1 (K)
- net EXP4: now reaches R36.2
- net EXP4: now also J4.4 (Pin_4)
- net EXP3: now reaches R35.2
- net EXP3: now also J4.5 (Pin_5)
- net EXP2: now reaches R34.2
- net EXP2: now also Q10.1 (G), R26.2, J4.3 (Pin_3)
- net EXP1: now reaches R33.2
- net EXP1: now also J4.6 (Pin_6)
- net EXP0: now reaches R32.2
- net EXP0: now also J3.1 (Pin_1)
- net at R40.2: now also D8.1 (K)
- net at Q10.3 (D): now also J9.2 (Pin_2); no longer J9.1 (Pin_1)
- net at D2.1 (K): no longer R29.2
- net at R8.2: now also D13.1 (K)
- net at Q6.3 (D): now also J7.2 (Pin_2), Q3.3 (D), Q5.3 (D)
- net at Q1.3 (D), Q2.3 (D), Q4.3 (D): now also J6.2 (Pin_2); no longer J6.1 (Pin_1)
- net GND_EB renamed GND1
- net GND1: now also J6.1 (Pin_1), J7.1 (Pin_1), J9.1 (Pin_1), R26.1, R29.1; no longer R12.2, R26.2
- net PB0 renamed PA5
- net PA5: now also U3.15 (PA5)
- net PC9 renamed PA8
- net PA8: now also U3.29 (PA8)
- removed net PWM2_E3: Q10.1 (G), R26.1
- net PWM3_E3: no longer names the net of Q6.1 (G)
- net PWM3_E3: now also R12.2; no longer R12.1
- removed net V_PWM_EB: J6.2 (Pin_2), J7.2 (Pin_2), J9.2 (Pin_2)
- net V_SERVO renamed V_EXP
- net V_EXP: now also J17.3 (Pin_3), J18.3 (Pin_3), J19.3 (Pin_3), J20.3 (Pin_3), J21.3 (Pin_3), J22.3 (Pin_3), D7.2 (A), J3.3 (Pin_3), J4.2 (Pin_2), JP1.2 (B)
- new net: D7.1 (K), R25.1
- new net PB12: U3.25 (PB12), U7.14 (PDN_UART)
Other:
- note added: "30V max"
- note added: "ADC, PWM, MISO"
- note added: "ADC, PWM, MOSI"
- note added: "ADC, PWM, SCK, not FT"
- note added: "ADC, SSEL, not FT"
- note added: "ENDSTOPS/SERVOS\n"
- note added: "EXPANSION BOARD - PRINTER"
- note added: "Extended parts:\nSTM32F411CEU6\nTMC2208-LA-T\n0805W8F250LT5F\nOVZ101M1ETR-0608\nSKRKAEE020\nCH912LSR"
- note added: "For defualt pins: https://github.com/stm32duino/Arduino_Tools/blob/master/src/genpinmap/Arduino/STM32F4/STM32F411C(C-E)Ux/PeripheralPins.c"
- note added: "PA3"
- note added: "PA4"
- note added: "PA5"
- note added: "PA6"
- note added: "PA7"
- note added: "PWM outputs are open drain!"
- note added: "PWM, ADC"
- note added: "PWM, RX"
- note added: "PWM, SCL"
- note added: "PWM, SDA"
- note added: "PWM, TX"
- note added: "UFQFPN-48_EP_7.0x7.0x0.5P"
- note added: "Used pin inputs are 5V tolerant!"
- note added: "ground loop prevention"
- note removed: "10A"
- note removed: "ENDSTOPS\n"
- note removed: "EXPANSION BOARD"
- note removed: "Extended parts:\nSTM32F411RCT6\nTMC2208-LA-T\n1206W4F250LT5E\nOVZ101M1ETR-0608\nSKRKAEE020\nCH912LSR"
- note removed: "For defualt pins: https://github.com/stm32duino/Arduino_Tools/blob/master/src/genpinmap/Arduino/STM32F4/STM32F411R(C-E)Tx/PeripheralPins.c"
- note removed: "I2C1_SCL, PWM"
- note removed: "I2C1_SDA, PWM"
- note removed: "I2C2_SCL, PWM"
- note removed: "I2C2_SDA, PWM"
- note removed: "LQFP-64_10.0x10.0x0.5P"
- note removed: "SERVOS"
- note removed: "SOD-123"
- note removed: "UART"
- note removed: "UART1"
- note removed: "Vmax=30V"
- note removed: "separate gnd\nto prevent\nground loops"
- moved on the sheet: C12, C19, C20, C21, C22, C23, C24, C25, C26, C7, C8, D2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

Commit message: working version with mosfets
Parts:
- J1: LCSC (none) -> C165948
Changed lines of the file:
@@
 F 2 "Connector_USB:USB_C_Receptacle_HRO_TYPE-C-31-M-12" H 2000 3400 50  0001 C CNN
 F 3 "https://www.usb.org/sites/default/files/documents/usb_type-c.zip" H 2000 3400 50  0001 C CNN
+F 4 "C165948" H 1850 3400 50  0001 C CNN "LCSC"
 	1    1850 3400
 	1    0    0    -1

Commit message: final, ordered
Parts:
- removed C25, C26: 4.7uF 10V, Capacitor_SMD:C_0402_1005Metric, symbol Device:C
- removed D3, D8: Yellow, LED_SMD:LED_0603_1608Metric, symbol Device:LED
- removed J16: ADC_HB, Connector_JST:JST_PH_B2B-PH-K_1x02_P2.00mm_Vertical, symbol Connector_Generic:Conn_01x02
- removed J29: ADC_E, Connector_JST:JST_PH_B2B-PH-K_1x02_P2.00mm_Vertical, symbol Connector_Generic:Conn_01x02
- removed J6: PWM_E, Connector_AMASS:AMASS_XT30U-F_1x02_P5.0mm_Vertical, symbol Connector_Generic:Conn_01x02
- removed J7: PWM_HB, Connector_AMASS:AMASS_XT30U-F_1x02_P5.0mm_Vertical, symbol Connector_Generic:Conn_01x02
- removed J9: PWM_FAN, Connector_JST:JST_PH_B2B-PH-K_1x02_P2.00mm_Vertical, symbol Connector_Generic:Conn_01x02
- removed Q1, Q10, Q2, Q3, Q4, Q5, Q6: AO3400A, Package_TO_SOT_SMD:SOT-23W, symbol Transistor_FET:2N7002
- removed R1, R2, R26: 330k, Resistor_SMD:R_0402_1005Metric, symbol Device:R
- removed R10, R11, R12, R29, R5, R6, R9: 330R, Resistor_SMD:R_0402_1005Metric, symbol Device:R
- removed R31, R37, R39, R40: 4.7k, Resistor_SMD:R_0402_1005Metric, symbol Device:R
Connections:
- net EXP0: no longer names the net of J3.1 (Pin_1), R32.2
- net EXP1: no longer names the net of J4.6 (Pin_6), R33.2
- net EXP2: no longer names the net of J4.3 (Pin_3), R34.2
- net EXP3: no longer names the net of J4.5 (Pin_5), R35.2
- net EXP4: no longer names the net of J4.4 (Pin_4), R36.2
Other:
- note removed: "0402WGF3303TCE\n0402"
- note removed: "0402WGF4701TCE\n0402"
- note removed: "15A"
- note removed: "30V max"
- note removed: "5A"
- note removed: "EXPANSION BOARD - PRINTER"
- note removed: "PA3"
- note removed: "PA4"
- note removed: "PA5"
- note removed: "PA6"
- note removed: "PA7"
- note removed: "PWM outputs are open drain!"
- note removed: "ground loop prevention"
- moved on the sheet: C27, C52, C68, D10, D11, D12, J3, J30, J31, J32, J4, R32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
